File: field-ambience-current/kicad/pi.kicad_sch (KiCad schematic)
At the start: 5 parts, among them J2 Pi Zero 2 W GPIO Header 2x20 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

Commit message: bom: stock/price check of all LCSC parts; swap R1 to Basic
Verified all 23 distinct LCSC numbers via jlcsearch (2026-05-29):
- 22/23 resolve cleanly; ~$3.62 SMT component cost per board.
- R1 was the only accidental Extended part (Yageo RC0603FR-071KL/C22548).
  Swapped to Uni Royal 0603WAF1001T5E/C21190 — same family as every other
  resistor, JLC Basic, 15.8M stock. No extended-part setup fee.

Flagged for the user (no blind change made):
- J8 jack C2884109 not in parts DB — confirm against the real purchased
  part before order (SMD candidate C431535). Tied to footprint check B0b.
- U2 MCP23017 C506653 stock only 357 — fine for one proto, watch for order.

MEINE_TODO Abschnitt 0 updated with the full result.

https://claude.ai/code/session_01K5kLTFpDCCoYwx2dq6RkAv
Parts:
- R1: LCSC C22548 -> C21190; MPN RC0603FR-071KL -> 0603WAF1001T5E
Changed lines of the file:
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@@
       (property "Datasheet" "~" (at 119 113.49000000000001 0)
         (effects (font (size 1.27 1.27)) hide))
-      (property "MPN" "RC0603FR-071KL" (at 121.54 117.30000000000001 0)
+      (property "MPN" "0603WAF1001T5E" (at 121.54 117.30000000000001 0)
         (effects (font (size 1.27 1.27)) hide))
-      (property "LCSC" "C22548" (at 121.54 118.57000000000001 0)
+      (property "LCSC" "C21190" (at 121.54 118.57000000000001 0)
         (effects (font (size 1.27 1.27)) hide))
     (instances

Commit message: fix(bom): make entire BOM correctly JLC-orderable — 7 real part errors fixed
Verified every LCSC number against jlcsearch for existence, stock, AND that
it resolves to the intended value/package. Found 7 parts that would have
built WRONG or were unorderable:

CRITICAL value/package errors (LCSC pointed at the wrong part):
- R_VOL_L/R: C25092 = 22ohm 0402  -> C4184  (real 20k 0603, Basic).
  Was wrong value AND footprint; would have wrecked the PAM8403 input gain.
- R_LO_L/R:  C22962 = 220ohm       -> C23345 (real 22ohm 0603, Basic).
- R_BCK/LRCK/DOUT: C23138 = 330ohm -> C23140 (real 33ohm 0603, Basic).

Unorderable -> assigned real in-stock parts:
- J8 jack:  C2884109 (nonexistent) -> C431535 (PJ-320D SMD).
- C_BULK:   placeholder            -> C46550395 (1000uF 16V SMD D10x10.5).
- LED1:     no LCSC                -> C965818 (white 0805).
- R1:       C22548 Extended        -> C21190 Basic (prior commit).

Also aligned all MPN text to the actual LCSC part (Yageo text vs Uni Royal/
Samsung parts JLC ships) so the BOM is internally consistent.

Re-verified: 25 distinct LCSC, all in stock, ZERO value/package mismatches,
14 Basic / 11 Extended. SPEC §4 stale refs (C_BULK/J8/R_LO) updated.
MEINE_TODO Abschnitt 0 rewritten with the full orderability result.

Self-supply parts (Pico, OLED, speakers, Choc sockets, EC11, headers) keep
no LCSC by design — JLC cannot assemble those.

https://claude.ai/code/session_01K5kLTFpDCCoYwx2dq6RkAv
Parts:
- R_BCK, R_DOUT, R_LRCK: LCSC C23138 -> C23140; MPN RC0603FR-0733RL -> 0603WAF330JT5E
Changed lines of the file:
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@@
       (property "Datasheet" "~" (at 140.08 118.57000000000001 0)
         (effects (font (size 1.27 1.27)) hide))
-      (property "MPN" "RC0603FR-0733RL" (at 142.62 122.38000000000001 0)
+      (property "MPN" "0603WAF330JT5E" (at 142.62 122.38000000000001 0)
         (effects (font (size 1.27 1.27)) hide))
-      (property "LCSC" "C23138" (at 142.62 123.65 0)
+      (property "LCSC" "C23140" (at 142.62 123.65 0)
         (effects (font (size 1.27 1.27)) hide))
     (instances
@@
       (property "Datasheet" "~" (at 119.92 149.05 0)
         (effects (font (size 1.27 1.27)) hide))
-      (property "MPN" "RC0603FR-0733RL" (at 122.46000000000001 152.86 0)
+      (property "MPN" "0603WAF330JT5E" (at 122.46000000000001 152.86 0)
         (effects (font (size 1.27 1.27)) hide))
-      (property "LCSC" "C23138" (at 122.46000000000001 154.13000000000002 0)
+      (property "LCSC" "C23140" (at 122.46000000000001 154.13000000000002 0)
         (effects (font (size 1.27 1.27)) hide))
     (instances
@@
       (property "Datasheet" "~" (at 140.08 154.13 0)
         (effects (font (size 1.27 1.27)) hide))
-      (property "MPN" "RC0603FR-0733RL" (at 142.62 157.94 0)
+      (property "MPN" "0603WAF330JT5E" (at 142.62 157.94 0)
         (effects (font (size 1.27 1.27)) hide))
-      (property "LCSC" "C23138" (at 142.62 159.21 0)
+      (property "LCSC" "C23140" (at 142.62 159.21 0)
         (effects (font (size 1.27 1.27)) hide))
     (instances
