File: field-ambience-current/kicad/mcp.kicad_sch (KiCad schematic)
At the start: 45 parts, among them SW1 Cell 1 (2u Choc V2 Hot-Swap), SW10 Modifier CLEAR (12x12x7.3 SMD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, SW2 Cell 2 (2u Choc V2 Hot-Swap), SW3 Cell 3 (2u Choc V2 Hot-Swap), SW4 Cell 4 (2u Choc V2 Hot-Swap), SW5 Cell 5 (2u Choc V2 Hot-Swap), SW6 Modifier SHIFT (12x12x7.3 SMD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, SW7 Modifier HOLD (12x12x7.3 SMD-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, SW8 Modifier DRONE (12x12x7.3 SMD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, SW9 Modifier GENERATE (12x12x7.3 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

Commit message: pcb(bom): r12-B12 — 9 falsche LCSC-Codes via jlcsearch-Audit korrigiert + r12-B11 TPS-Package-Blocker
JLC-Pricing-Estimate-Run hat 9 falsche LCSC-Codes im Generator aufgedeckt.
Alle MPN-Strings waren korrekt, aber die zugewiesenen LCSC-Codes pointed
auf völlig andere Teile. Bei sofortiger JLC-Bestellung wäre der Prototyp
DOA gewesen (BAT_SENSE-Divider 130Ω/130Ω statt 100k/100k, Boost-FB 15Ω/0.21k
statt 200k/39k, alle LEDs nicht-existent, etc.).

Korrigierte Mappings (via jlcsearch-API-Verifikation):
- 100kΩ 0603 (R_BAT_DIV_TOP/BOT, R_VBUS_PD): C22796 → C25803 (Basic)
- 200kΩ 0603 (R23): C22810 → C25811 (Basic)
- 39kΩ 0603 (R24): C25090 → C23153 (Basic)
- 390Ω 0603 (R_LED6-15, R_LED_STATUS): C23289 → C23151 (Basic)
- MCP73831T-2ACI/OT (U7): C14879 → C424093 (Extended)
- DMG2305UX-7 (Q1): C147074 → C150470 (Extended)
- SWPA6045S2R2MT (L1): C32330 → C83455 (Extended)
- S2B-PH-SM4-TB SMD (J9): C146061 → C295747 (Extended)
- 0603 white LED (LED1, LED6-15): C72043 → C965808 XL-1608UWC-04 (Extended)

Neuer BLOCKER r12-B11: TPS61089-Package-Mismatch
SPEC §2.2 spezifiziert TPS61089RNSR (QFN-12 3×3mm), aber LCSC hat nur
TPS61089RNRR (VQFN-11 2×2.5mm HotRod, anderer Footprint + Pinout).
Generator markiert LCSC vorerst als "TBD-USER-SUPPLY-or-RNRR-refactor"
bis User-Decision. 3 Lösungswege in PCB_TODO r12-B11 dokumentiert
(RNRR-Refactor / RNSR-Konsignierung / Hand-Solder).

Side-Effekt: 4 der korrigierten Resistor-SKUs sind Basic (kein Extended-
Setup-Fee) → spart $12 bei 5-Boards. Extended-SKU-Count 23 → 19.

JLC-Cost-Estimate aktualisiert in CHANGELOG: 5 Prototyp-Boards ~$567
(JLC $294 + User-Supplied $272 + Battery/OLED/Choc/Pico/Speaker), per
Board ~$113. Bei 100 Stück ~$6884 (~$69/Board).

Generator/SPEC/PCB_TODO/CHANGELOG synchron. Analyzer-Status unverändert
(LCSC sind Metadata, keine Connectivity-Änderung).

https://claude.ai/code/session_01K5kLTFpDCCoYwx2dq6RkAv
Parts:
- LED1: LCSC C72043 -> C965808; MPN Generic warm-white 0603 -> XL-1608UWC-04 (warm-white 0603, Extended)
- LED10, LED11, LED12, LED13, LED14, LED15, LED6, LED7, LED8, LED9: LCSC C72043 -> C965808; MPN Generic warm-white/amber 0603 -> XL-1608UWC-04 (warm-white 0603, Extended)
- R_LED10, R_LED11, R_LED12, R_LED13, R_LED14, R_LED15, R_LED6, R_LED7, R_LED8, R_LED9, R_LED_STATUS: LCSC C23289 -> C23151
- R_VBUS_PD: LCSC C22796 -> C25803
Changed lines of the file:
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@@
       (property "MPN" "0603WAF1003T5E" (at 151.54 107.3 0)
         (effects (font (size 1.27 1.27)) hide))
-      (property "LCSC" "C22796" (at 151.54 108.57 0)
+      (property "LCSC" "C25803" (at 151.54 108.57 0)
         (effects (font (size 1.27 1.27)) hide))
     (instances
@@
       (property "MPN" "0603WAF3900T5E" (at 82.54 203.81 0)
         (effects (font (size 1.27 1.27)) hide))
-      (property "LCSC" "C23289" (at 82.54 205.08 0)
+      (property "LCSC" "C23151" (at 82.54 205.08 0)
         (effects (font (size 1.27 1.27)) hide))
     (instances
@@
       (property "Datasheet" "~" (at 87.62 200 0)
         (effects (font (size 1.27 1.27)) hide))
-      (property "MPN" "Generic warm-white/amber 0603" (at 90.16000000000001 203.81 0)
-        (effects (font (size 1.27 1.27)) hide))
-      (property "LCSC" "C72043" (at 90.16000000000001 205.08 0)
+      (property "MPN" "XL-1608UWC-04 (warm-white 0603, Extended)" (at 90.16000000000001 203.81 0)
+        (effects (font (size 1.27 1.27)) hide))
+      (property "LCSC" "C965808" (at 90.16000000000001 205.08 0)
         (effects (font (size 1.27 1.27)) hide))
     (instances
@@
       (property "MPN" "0603WAF3900T5E" (at 107.54 203.81 0)
         (effects (font (size 1.27 1.27)) hide))
-      (property "LCSC" "C23289" (at 107.54 205.08 0)
+      (property "LCSC" "C23151" (at 107.54 205.08 0)
         (effects (font (size 1.27 1.27)) hide))
     (instances
@@
       (property "Datasheet" "~" (at 112.62 200 0)
         (effects (font (size 1.27 1.27)) hide))
-      (property "MPN" "Generic warm-white/amber 0603" (at 115.16000000000001 203.81 0)
-        (effects (font (size 1.27 1.27)) hide))
-      (property "LCSC" "C72043" (at 115.16000000000001 205.08 0)
+      (property "MPN" "XL-1608UWC-04 (warm-white 0603, Extended)" (at 115.16000000000001 203.81 0)
+        (effects (font (size 1.27 1.27)) hide))
+      (property "LCSC" "C965808" (at 115.16000000000001 205.08 0)
         (effects (font (size 1.27 1.27)) hide))
     (instances
@@
       (property "MPN" "0603WAF3900T5E" (at 132.54 203.81 0)
         (effects (font (size 1.27 1.27)) hide))
-      (property "LCSC" "C23289" (at 132.54 205.08 0)
+      (property "LCSC" "C23151" (at 132.54 205.08 0)
         (effects (font (size 1.27 1.27)) hide))
     (instances
@@
       (property "Datasheet" "~" (at 137.62 200 0)
         (effects (font (size 1.27 1.27)) hide))
-      (property "MPN" "Generic warm-white/amber 0603" (at 140.16 203.81 0)
-        (effects (font (size 1.27 1.27)) hide))
-      (property "LCSC" "C72043" (at 140.16 205.08 0)
+      (property "MPN" "XL-1608UWC-04 (warm-white 0603, Extended)" (at 140.16 203.81 0)
+        (effects (font (size 1.27 1.27)) hide))
+      (property "LCSC" "C965808" (at 140.16 205.08 0)
         (effects (font (size 1.27 1.27)) hide))
     (instances
@@
       (property "MPN" "0603WAF3900T5E" (at 157.54 203.81 0)
         (effects (font (size 1.27 1.27)) hide))
-      (property "LCSC" "C23289" (at 157.54 205.08 0)
+      (property "LCSC" "C23151" (at 157.54 205.08 0)
         (effects (font (size 1.27 1.27)) hide))
     (instances
@@
       (property "Datasheet" "~" (at 162.62 200 0)
         (effects (font (size 1.27 1.27)) hide))
-      (property "MPN" "Generic warm-white/amber 0603" (at 165.16 203.81 0)
-        (effects (font (size 1.27 1.27)) hide))
-      (property "LCSC" "C72043" (at 165.16 205.08 0)
+      (property "MPN" "XL-1608UWC-04 (warm-white 0603, Extended)" (at 165.16 203.81 0)
+        (effects (font (size 1.27 1.27)) hide))
+      (property "LCSC" "C965808" (at 165.16 205.08 0)
         (effects (font (size 1.27 1.27)) hide))
     (instances
@@
       (property "MPN" "0603WAF3900T5E" (at 182.54 203.81 0)
         (effects (font (size 1.27 1.27)) hide))
-      (property "LCSC" "C23289" (at 182.54 205.08 0)
+      (property "LCSC" "C23151" (at 182.54 205.08 0)
         (effects (font (size 1.27 1.27)) hide))
     (instances
@@
       (property "Datasheet" "~" (at 187.62 200 0)
         (effects (font (size 1.27 1.27)) hide))
-      (property "MPN" "Generic warm-white/amber 0603" (at 190.16 203.81 0)
-        (effects (font (size 1.27 1.27)) hide))
-      (property "LCSC" "C72043" (at 190.16 205.08 0)
+      (property "MPN" "XL-1608UWC-04 (warm-white 0603, Extended)" (at 190.16 203.81 0)
+        (effects (font (size 1.27 1.27)) hide))
+      (property "LCSC" "C965808" (at 190.16 205.08 0)
         (effects (font (size 1.27 1.27)) hide))
     (instances
@@
       (property "MPN" "0603WAF3900T5E" (at 82.54 218.81 0)
         (effects (font (size 1.27 1.27)) hide))
-      (property "LCSC" "C23289" (at 82.54 220.08 0)
+      (property "LCSC" "C23151" (at 82.54 220.08 0)
         (effects (font (size 1.27 1.27)) hide))
     (instances
@@
       (property "Datasheet" "~" (at 87.62 215 0)
         (effects (font (size 1.27 1.27)) hide))
-      (property "MPN" "Generic warm-white/amber 0603" (at 90.16000000000001 218.81 0)
-        (effects (font (size 1.27 1.27)) hide))
-      (property "LCSC" "C72043" (at 90.16000000000001 220.08 0)
+      (property "MPN" "XL-1608UWC-04 (warm-white 0603, Extended)" (at 90.16000000000001 218.81 0)
+        (effects (font (size 1.27 1.27)) hide))
+      (property "LCSC" "C965808" (at 90.16000000000001 220.08 0)
         (effects (font (size 1.27 1.27)) hide))
     (instances
@@
       (property "MPN" "0603WAF3900T5E" (at 107.54 218.81 0)
         (effects (font (size 1.27 1.27)) hide))
-      (property "LCSC" "C23289" (at 107.54 220.08 0)
+      (property "LCSC" "C23151" (at 107.54 220.08 0)
         (effects (font (size 1.27 1.27)) hide))
     (instances
@@
       (property "Datasheet" "~" (at 112.62 215 0)
         (effects (font (size 1.27 1.27)) hide))
-      (property "MPN" "Generic warm-white/amber 0603" (at 115.16000000000001 218.81 0)
-        (effects (font (size 1.27 1.27)) hide))
-      (property "LCSC" "C72043" (at 115.16000000000001 220.08 0)
+      (property "MPN" "XL-1608UWC-04 (warm-white 0603, Extended)" (at 115.16000000000001 218.81 0)
+        (effects (font (size 1.27 1.27)) hide))
+      (property "LCSC" "C965808" (at 115.16000000000001 220.08 0)
         (effects (font (size 1.27 1.27)) hide))
     (instances
@@
       (property "MPN" "0603WAF3900T5E" (at 132.54 218.81 0)
         (effects (font (size 1.27 1.27)) hide))
-      (property "LCSC" "C23289" (at 132.54 220.08 0)
+      (property "LCSC" "C23151" (at 132.54 220.08 0)
         (effects (font (size 1.27 1.27)) hide))
     (instances
@@
       (property "Datasheet" "~" (at 137.62 215 0)
         (effects (font (size 1.27 1.27)) hide))
-      (property "MPN" "Generic warm-white/amber 0603" (at 140.16 218.81 0)
-        (effects (font (size 1.27 1.27)) hide))
-      (property "LCSC" "C72043" (at 140.16 220.08 0)
+      (property "MPN" "XL-1608UWC-04 (warm-white 0603, Extended)" (at 140.16 218.81 0)
+        (effects (font (size 1.27 1.27)) hide))
+      (property "LCSC" "C965808" (at 140.16 220.08 0)
         (effects (font (size 1.27 1.27)) hide))
     (instances
@@
       (property "MPN" "0603WAF3900T5E" (at 157.54 218.81 0)
         (effects (font (size 1.27 1.27)) hide))
-      (property "LCSC" "C23289" (at 157.54 220.08 0)
+      (property "LCSC" "C23151" (at 157.54 220.08 0)
         (effects (font (size 1.27 1.27)) hide))
     (instances
@@
       (property "Datasheet" "~" (at 162.62 215 0)
         (effects (font (size 1.27 1.27)) hide))
-      (property "MPN" "Generic warm-white/amber 0603" (at 165.16 218.81 0)
-        (effects (font (size 1.27 1.27)) hide))
-      (property "LCSC" "C72043" (at 165.16 220.08 0)
+      (property "MPN" "XL-1608UWC-04 (warm-white 0603, Extended)" (at 165.16 218.81 0)
+        (effects (font (size 1.27 1.27)) hide))
+      (property "LCSC" "C965808" (at 165.16 220.08 0)
         (effects (font (size 1.27 1.27)) hide))
     (instances
@@
       (property "MPN" "0603WAF3900T5E" (at 182.54 218.81 0)
         (effects (font (size 1.27 1.27)) hide))
-      (property "LCSC" "C23289" (at 182.54 220.08 0)
+      (property "LCSC" "C23151" (at 182.54 220.08 0)
         (effects (font (size 1.27 1.27)) hide))
     (instances
@@
       (property "Datasheet" "~" (at 187.62 215 0)
         (effects (font (size 1.27 1.27)) hide))
-      (property "MPN" "Generic warm-white/amber 0603" (at 190.16 218.81 0)
-        (effects (font (size 1.27 1.27)) hide))
-      (property "LCSC" "C72043" (at 190.16 220.08 0)
+      (property "MPN" "XL-1608UWC-04 (warm-white 0603, Extended)" (at 190.16 218.81 0)
+        (effects (font (size 1.27 1.27)) hide))
+      (property "LCSC" "C965808" (at 190.16 220.08 0)
         (effects (font (size 1.27 1.27)) hide))
     (instances
@@
       (property "MPN" "0603WAF3900T5E" (at 132.54 233.81 0)
         (effects (font (size 1.27 1.27)) hide))
-      (property "LCSC" "C23289" (at 132.54 235.08 0)
+      (property "LCSC" "C23151" (at 132.54 235.08 0)
         (effects (font (size 1.27 1.27)) hide))
     (instances
@@
       (property "Datasheet" "~" (at 137.62 230.0 0)
         (effects (font (size 1.27 1.27)) hide))
-      (property "MPN" "Generic warm-white 0603" (at 140.16 233.81 0)
-        (effects (font (size 1.27 1.27)) hide))
-      (property "LCSC" "C72043" (at 140.16 235.08 0)
-        (effects (font (size 1.27 1.27)) hide))
-    (instances
+      (property "MPN" "XL-1608UWC-04 (warm-white 0603, Extended)" (at 140.16 233.81 0)
+        (effects (font (size 1.27 1.27)) hide))
+      (property "LCSC" "C965808" (at 140.16 235.08 0)
+        (effects (font (size 1.27 1.27)) hide))
+    (instances
