File: field-ambience-current/kicad/mcp.kicad_sch (KiCad schematic)
At the start: 48 parts, among them SW10 Modifier CLEAR (12x12x7.3 SMD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, SW6 Modifier SHIFT (12x12x7.3 SMD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, SW7 Modifier HOLD (12x12x7.3 SMD-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, SW8 Modifier DRONE (12x12x7.3 SMD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, SW9 Modifier GENERATE (12x12x7.3 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, U2 MCP23017-E/SS (I/O-Expander), U6 PCA9685PW (16-Ch I²C PWM LED-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

Commit message: pcb(r18.20b): Sourcing-Fills — alle JLC-bestückbaren TBD-LCSC geschlossen
Sourcing-Agent lieferte verifizierte in-Stock-LCSC für alle r18.20-TBDs:
- C_HSE1/2:  C107045 (Yageo 27pF C0G/NP0 0603, JLC Basic, ~834k Stock)
- C_BULK:    C444831 (Kyocera AVX TPSE477K010R0100, 470µF/10V Polymer Case-E)
- C_BULK2:   C2880380 (Taiyo Yuden 100µF/10V 1210)
- LED gelb:  C2287 (Hubei KENTO KT-0603Y, Vf 2.4V) — Hold + 5 Cell
- LED grün:  C12624 (Hubei KENTO KT-0603G pure-green, Vf 3.1V) — Shift + 5 Cell

Engineering-Flag 1: "220µF/10V/1210 existiert nicht" (220µF nur bis 6.3V im
1210). Statt 220µF/6.3V (am 5V-Rail auf ~70-110µF derated) → 100µF/10V mit
echtem Headroom. Effektiv-Bulk vergleichbar, audit-sauber.

Engineering-Flag 2: <25mΩ-Flach-Polymer (Panasonic SVPF/Kemet T520) bei LCSC
nicht lagernd. Bester JLC-Flach-Polymer C444831 (100mΩ). Verfehlt 10mΩ-Ziel,
aber paralleler 100µF-MLCC (~5mΩ) dominiert Transient-Impedanz → Bulk-ESR
unkritisch. Footprint Case-D→Case-E (7343-43, 4.3mm, passt in 8mm-Top-Zone).

Beifang: BOM_MASTER §9 sagte "220Ω LED-R", Generator sagt 390Ω (an +5V-Anode
→ LED → PCA9685-Sink). 5V/390Ω: gelb 6.7mA, grün 4.9mA — beide im 2-8mA-
Fenster, Wert bleibt. BOM_MASTER korrigiert.

Verifizierung: 8/8 paren-balanced, 0 TBD-VERIFY-Leftovers in power_tree+mcp,
LED gelb ×6 + grün ×6, Firmware 13/13 PASS.

Files: generate_kicad_project.py (5 Fills), 3 Sheets regen, BOM_MASTER,
ADR-0011 (ESR-Realität), CHANGELOG, PROJECT_QUALITY BOM 9.5→10, Readiness 6.5→7.

https://claude.ai/code/session_01K5kLTFpDCCoYwx2dq6RkAv
Parts:
- LED11G, LED12G, LED13G, LED14G, LED15G, LED6: LCSC TBD-VERIFY (JLC-Stock gruen 0603) -> C12624; MPN XL-1608UGC-04 (green 0603, XINGLIGHT-Serie) -> KT-0603G (Hubei KENTO, pure green 525nm 0603, Vf 3.1V)
- LED11Y, LED12Y, LED13Y, LED14Y, LED15Y, LED7: LCSC TBD-VERIFY (JLC-Stock gelb 0603) -> C2287; MPN XL-1608UYC-04 (yellow 0603, XINGLIGHT-Serie) -> KT-0603Y (Hubei KENTO, yellow 0603, Vf 2.4V)
Changed lines of the file:
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@@
       (property "Datasheet" "~" (at 87.62 200 0)
         (effects (font (size 1.27 1.27)) hide))
-      (property "MPN" "XL-1608UGC-04 (green 0603, XINGLIGHT-Serie)" (at 90.16000000000001 203.81 0)
-        (effects (font (size 1.27 1.27)) hide))
-      (property "LCSC" "TBD-VERIFY (JLC-Stock gruen 0603)" (at 90.16000000000001 205.08 0)
+      (property "MPN" "KT-0603G (Hubei KENTO, pure green 525nm 0603, Vf 3.1V)" (at 90.16000000000001 203.81 0)
+        (effects (font (size 1.27 1.27)) hide))
+      (property "LCSC" "C12624" (at 90.16000000000001 205.08 0)
         (effects (font (size 1.27 1.27)) hide))
     (instances
@@
       (property "Datasheet" "~" (at 112.62 200 0)
         (effects (font (size 1.27 1.27)) hide))
-      (property "MPN" "XL-1608UYC-04 (yellow 0603, XINGLIGHT-Serie)" (at 115.16000000000001 203.81 0)
-        (effects (font (size 1.27 1.27)) hide))
-      (property "LCSC" "TBD-VERIFY (JLC-Stock gelb 0603)" (at 115.16000000000001 205.08 0)
+      (property "MPN" "KT-0603Y (Hubei KENTO, yellow 0603, Vf 2.4V)" (at 115.16000000000001 203.81 0)
+        (effects (font (size 1.27 1.27)) hide))
+      (property "LCSC" "C2287" (at 115.16000000000001 205.08 0)
         (effects (font (size 1.27 1.27)) hide))
     (instances
@@
       (property "Datasheet" "~" (at 87.62 215 0)
         (effects (font (size 1.27 1.27)) hide))
-      (property "MPN" "XL-1608UYC-04 (yellow 0603, XINGLIGHT-Serie)" (at 90.16000000000001 218.81 0)
-        (effects (font (size 1.27 1.27)) hide))
-      (property "LCSC" "TBD-VERIFY (JLC-Stock gelb 0603)" (at 90.16000000000001 220.08 0)
+      (property "MPN" "KT-0603Y (Hubei KENTO, yellow 0603, Vf 2.4V)" (at 90.16000000000001 218.81 0)
+        (effects (font (size 1.27 1.27)) hide))
+      (property "LCSC" "C2287" (at 90.16000000000001 220.08 0)
         (effects (font (size 1.27 1.27)) hide))
     (instances
@@
       (property "Datasheet" "~" (at 87.62 228 0)
         (effects (font (size 1.27 1.27)) hide))
-      (property "MPN" "XL-1608UGC-04 (green 0603, XINGLIGHT-Serie)" (at 90.16000000000001 231.81 0)
-        (effects (font (size 1.27 1.27)) hide))
-      (property "LCSC" "TBD-VERIFY (JLC-Stock gruen 0603)" (at 90.16000000000001 233.08 0)
+      (property "MPN" "KT-0603G (Hubei KENTO, pure green 525nm 0603, Vf 3.1V)" (at 90.16000000000001 231.81 0)
+        (effects (font (size 1.27 1.27)) hide))
+      (property "LCSC" "C12624" (at 90.16000000000001 233.08 0)
         (effects (font (size 1.27 1.27)) hide))
     (instances
@@
       (property "Datasheet" "~" (at 112.62 215 0)
         (effects (font (size 1.27 1.27)) hide))
-      (property "MPN" "XL-1608UYC-04 (yellow 0603, XINGLIGHT-Serie)" (at 115.16000000000001 218.81 0)
-        (effects (font (size 1.27 1.27)) hide))
-      (property "LCSC" "TBD-VERIFY (JLC-Stock gelb 0603)" (at 115.16000000000001 220.08 0)
+      (property "MPN" "KT-0603Y (Hubei KENTO, yellow 0603, Vf 2.4V)" (at 115.16000000000001 218.81 0)
+        (effects (font (size 1.27 1.27)) hide))
+      (property "LCSC" "C2287" (at 115.16000000000001 220.08 0)
         (effects (font (size 1.27 1.27)) hide))
     (instances
@@
       (property "Datasheet" "~" (at 112.62 228 0)
         (effects (font (size 1.27 1.27)) hide))
-      (property "MPN" "XL-1608UGC-04 (green 0603, XINGLIGHT-Serie)" (at 115.16000000000001 231.81 0)
-        (effects (font (size 1.27 1.27)) hide))
-      (property "LCSC" "TBD-VERIFY (JLC-Stock gruen 0603)" (at 115.16000000000001 233.08 0)
+      (property "MPN" "KT-0603G (Hubei KENTO, pure green 525nm 0603, Vf 3.1V)" (at 115.16000000000001 231.81 0)
+        (effects (font (size 1.27 1.27)) hide))
+      (property "LCSC" "C12624" (at 115.16000000000001 233.08 0)
         (effects (font (size 1.27 1.27)) hide))
     (instances
@@
       (property "Datasheet" "~" (at 137.62 215 0)
         (effects (font (size 1.27 1.27)) hide))
-      (property "MPN" "XL-1608UYC-04 (yellow 0603, XINGLIGHT-Serie)" (at 140.16 218.81 0)
-        (effects (font (size 1.27 1.27)) hide))
-      (property "LCSC" "TBD-VERIFY (JLC-Stock gelb 0603)" (at 140.16 220.08 0)
+      (property "MPN" "KT-0603Y (Hubei KENTO, yellow 0603, Vf 2.4V)" (at 140.16 218.81 0)
+        (effects (font (size 1.27 1.27)) hide))
+      (property "LCSC" "C2287" (at 140.16 220.08 0)
         (effects (font (size 1.27 1.27)) hide))
     (instances
@@
       (property "Datasheet" "~" (at 137.62 228 0)
         (effects (font (size 1.27 1.27)) hide))
-      (property "MPN" "XL-1608UGC-04 (green 0603, XINGLIGHT-Serie)" (at 140.16 231.81 0)
-        (effects (font (size 1.27 1.27)) hide))
-      (property "LCSC" "TBD-VERIFY (JLC-Stock gruen 0603)" (at 140.16 233.08 0)
+      (property "MPN" "KT-0603G (Hubei KENTO, pure green 525nm 0603, Vf 3.1V)" (at 140.16 231.81 0)
+        (effects (font (size 1.27 1.27)) hide))
+      (property "LCSC" "C12624" (at 140.16 233.08 0)
         (effects (font (size 1.27 1.27)) hide))
     (instances
@@
       (property "Datasheet" "~" (at 162.62 215 0)
         (effects (font (size 1.27 1.27)) hide))
-      (property "MPN" "XL-1608UYC-04 (yellow 0603, XINGLIGHT-Serie)" (at 165.16 218.81 0)
-        (effects (font (size 1.27 1.27)) hide))
-      (property "LCSC" "TBD-VERIFY (JLC-Stock gelb 0603)" (at 165.16 220.08 0)
+      (property "MPN" "KT-0603Y (Hubei KENTO, yellow 0603, Vf 2.4V)" (at 165.16 218.81 0)
+        (effects (font (size 1.27 1.27)) hide))
+      (property "LCSC" "C2287" (at 165.16 220.08 0)
         (effects (font (size 1.27 1.27)) hide))
     (instances
@@
       (property "Datasheet" "~" (at 162.62 228 0)
         (effects (font (size 1.27 1.27)) hide))
-      (property "MPN" "XL-1608UGC-04 (green 0603, XINGLIGHT-Serie)" (at 165.16 231.81 0)
-        (effects (font (size 1.27 1.27)) hide))
-      (property "LCSC" "TBD-VERIFY (JLC-Stock gruen 0603)" (at 165.16 233.08 0)
+      (property "MPN" "KT-0603G (Hubei KENTO, pure green 525nm 0603, Vf 3.1V)" (at 165.16 231.81 0)
+        (effects (font (size 1.27 1.27)) hide))
+      (property "LCSC" "C12624" (at 165.16 233.08 0)
         (effects (font (size 1.27 1.27)) hide))
     (instances
@@
       (property "Datasheet" "~" (at 187.62 215 0)
         (effects (font (size 1.27 1.27)) hide))
-      (property "MPN" "XL-1608UYC-04 (yellow 0603, XINGLIGHT-Serie)" (at 190.16 218.81 0)
-        (effects (font (size 1.27 1.27)) hide))
-      (property "LCSC" "TBD-VERIFY (JLC-Stock gelb 0603)" (at 190.16 220.08 0)
+      (property "MPN" "KT-0603Y (Hubei KENTO, yellow 0603, Vf 2.4V)" (at 190.16 218.81 0)
+        (effects (font (size 1.27 1.27)) hide))
+      (property "LCSC" "C2287" (at 190.16 220.08 0)
         (effects (font (size 1.27 1.27)) hide))
     (instances
@@
       (property "Datasheet" "~" (at 187.62 228 0)
         (effects (font (size 1.27 1.27)) hide))
-      (property "MPN" "XL-1608UGC-04 (green 0603, XINGLIGHT-Serie)" (at 190.16 231.81 0)
-        (effects (font (size 1.27 1.27)) hide))
-      (property "LCSC" "TBD-VERIFY (JLC-Stock gruen 0603)" (at 190.16 233.08 0)
-        (effects (font (size 1.27 1.27)) hide))
-    (instances
+      (property "MPN" "KT-0603G (Hubei KENTO, pure green 525nm 0603, Vf 3.1V)" (at 190.16 231.81 0)
+        (effects (font (size 1.27 1.27)) hide))
+      (property "LCSC" "C12624" (at 190.16 233.08 0)
+        (effects (font (size 1.27 1.27)) hide))
+    (instances
