File: field-ambience-current/kicad/mcp.kicad_sch (KiCad schematic)
At the start: 73 parts, among them SW1 Cell 1 digital trigger (Kailh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, SW10 Modifier CLEAR (HX B3F-4055 T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, SW2 Cell 2 digital trigger (Kailh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, SW3 Cell 3 digital trigger (Kailh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, SW4 Cell 4 digital trigger (Kailh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, SW5 Cell 5 digital trigger (Kailh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, SW6 Modifier SHIFT (HX B3F-4055 T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, SW7 Modifier HOLD (HX B3F-4055 TH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, SW8 Modifier DRONE (HX B3F-4055 T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, SW9 Modifier GENERATE (HX B3F-405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, U10 PCA9685PW #2 (16-Ch I²C PWM, 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, U2 MCP23017-E/SS (I/O-Expander), U6 PCA9685PW (16-Ch I²C PWM LED-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

Commit message: fix(pcb): geometric pin-level ERC — 7 copper shorts, 4 open circuits, boost loop instability (r18.80) (#92)
Headless geometric ERC (every pin anchor vs every wire segment, union-find
net build, hier-label/root-pin matching) over all 7 sheets found 12 real
defects; each verified in generator source and fixed there.

Copper shorts (pin/label anchors landing on foreign wires):
- power_tree: USB D+ AND D- hard-shorted to +5V — the U5 LDO block sat in
  the USB data corridor (EN pin on the DP wire, IN pin on the DM wire,
  rail drop overlapping the ESD VBUS wire). Block moved to (130,130).
- mcp: I2C_SCL shorted to GND — C5's GND pin landed exactly on the SCL
  wire (VDD pin 9 and SCL pin 12 are exactly 3 grid rows = 7.62mm apart,
  the cap's pin pitch). Entire I2C bus (U2+U6+U10) was dead. C5/C5b moved.
- audio: PCM_XSMT and I2S_LRCK shorted to GND (same 7.62mm trap, C8a/C8b
  and C_LDOO) — DAC permanently muted / no word clock. Caps flipped up.
- stm32: BOOT0 permanently HIGH twice over (+3V3 flag placed on the BOOT0
  node point; SW_BOOT wire drawn through its own pin-2 anchor) — MCU would
  always enter the ROM bootloader, never firmware.
- stm32: VDDA copper-tied to VDD (pin-21 stub drawn through the VDD pin-100
  anchor), bypassing FB2.
- battery: U8_SW_NODE label sat on the SW/BOOT wire crossing, merging the
  bootstrap net with the switch node (C_BOOT ineffective).

Open circuits:
- lcd: J3 LCD header — all 8 pins floating (wiring assumed KiCad-standard
  pins at -5.08 left; custom lib has pins at +3.81 right). J3 rotated 180.
- stm32: J4 SWD header — all 3 pins floating (same assumption). Board was
  unprogrammable.
- stm32: FB2 rotated 90 off its wires — both pins floating (VDDA had no
  intended supply path).
- stm32: lib_symbols entry lacked the MCU: prefix — KiCad cannot resolve
  U1 at all (exact lib_id match required).

Boost control loop (TPS61089, TI SLVSD38C eqs 15/17/18, validated by
reproducing TI's own 9V/2A reference values):
- R_COMP 22k -> 6.2k (n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
Parts:
- C_PCA2_VDD, C_PCA_VDD: MPN CL21A106KOQNNNG-class -> CL21A106KAYNNNE
- C_PCA2_VDD_HF, C_PCA_VDD_HF: MPN CL10B104KO8NNNC-class -> CC0603KRX7R9BB104
Connections:
- no-connect marks 0 -> 8
Other:
- moved on the sheet: C5, C5b
Changed lines of the file:
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@@
       (project "field_ambience"
         (path "/ae4d8abd-ab57-48bd-a18a-f37b38917ad2" (reference "#PWR_U2_VDD") (unit 1)))))
-  (symbol (lib_id "Device:C") (at 108 117.62 0) (unit 1)
-    (in_bom yes) (on_board yes) (dnp no)
-      (property "Reference" "C5" (at 110.54 115.08 0)
-        (effects (font (size 1.27 1.27))))
-      (property "Value" "100nF X7R 0603 (VDD HF)" (at 110.54 118.89 0)
-        (effects (font (size 1.27 1.27))))
-      (property "Footprint" "Capacitor_SMD:C_0603_1608Metric" (at 108 117.62 0)
-        (effects (font (size 1.27 1.27)) hide))
-      (property "Datasheet" "~" (at 108 117.62 0)
-        (effects (font (size 1.27 1.27)) hide))
-      (property "MPN" "CC0603KRX7R9BB104" (at 110.54 121.43 0)
-        (effects (font (size 1.27 1.27)) hide))
-      (property "LCSC" "C14663" (at 110.54 122.7 0)
+  (symbol (lib_id "Device:C") (at 93 117.62 0) (unit 1)
+    (in_bom yes) (on_board yes) (dnp no)
+      (property "Reference" "C5" (at 95.54 115.08 0)
+        (effects (font (size 1.27 1.27))))
+      (property "Value" "100nF X7R 0603 (VDD HF)" (at 95.54 118.89 0)
+        (effects (font (size 1.27 1.27))))
+      (property "Footprint" "Capacitor_SMD:C_0603_1608Metric" (at 93 117.62 0)
+        (effects (font (size 1.27 1.27)) hide))
+      (property "Datasheet" "~" (at 93 117.62 0)
+        (effects (font (size 1.27 1.27)) hide))
+      (property "MPN" "CC0603KRX7R9BB104" (at 95.54 121.43 0)
+        (effects (font (size 1.27 1.27)) hide))
+      (property "LCSC" "C14663" (at 95.54 122.7 0)
         (effects (font (size 1.27 1.27)) hide))
     (instances
       (project "field_ambience"
         (path "/ae4d8abd-ab57-48bd-a18a-f37b38917ad2" (reference "C5") (unit 1)))))
-  (symbol (lib_id "Power:GND") (at 108 123.81 270) (unit 1)
-    (in_bom yes) (on_board yes) (dnp no)
-      (property "Reference" "#PWR_C5" (at 110.54 121.27 0)
-        (effects (font (size 1.27 1.27))))
-      (property "Value" "GND" (at 110.54 125.08 0)
-        (effects (font (size 1.27 1.27))))
-      (property "Footprint" "" (at 108 123.81 0)
-        (effects (font (size 1.27 1.27)) hide))
-      (property "Datasheet" "~" (at 108 123.81 0)
+  (symbol (lib_id "Power:GND") (at 93 123.81 270) (unit 1)
+    (in_bom yes) (on_board yes) (dnp no)
+      (property "Reference" "#PWR_C5" (at 95.54 121.27 0)
+        (effects (font (size 1.27 1.27))))
+      (property "Value" "GND" (at 95.54 125.08 0)
+        (effects (font (size 1.27 1.27))))
+      (property "Footprint" "" (at 93 123.81 0)
+        (effects (font (size 1.27 1.27)) hide))
+      (property "Datasheet" "~" (at 93 123.81 0)
         (effects (font (size 1.27 1.27)) hide))
     (instances
       (project "field_ambience"
         (path "/ae4d8abd-ab57-48bd-a18a-f37b38917ad2" (reference "#PWR_C5") (unit 1)))))
-  (symbol (lib_id "Device:C") (at 103 117.62 0) (unit 1)
-    (in_bom yes) (on_board yes) (dnp no)
-      (property "Reference" "C5b" (at 105.54 115.08 0)
-        (effects (font (size 1.27 1.27))))
-      (property "Value" "10nF X7R 0603 (VDD HF²)" (at 105.54 118.89 0)
-        (effects (font (size 1.27 1.27))))
-      (property "Footprint" "Capacitor_SMD:C_0603_1608Metric" (at 103 117.62 0)
-        (effects (font (size 1.27 1.27)) hide))
-      (property "Datasheet" "~" (at 103 117.62 0)
-        (effects (font (size 1.27 1.27)) hide))
-      (property "MPN" "0603B103K500NT" (at 105.54 121.43 0)
-        (effects (font (size 1.27 1.27)) hide))
-      (property "LCSC" "C57112" (at 105.54 122.7 0)
+  (symbol (lib_id "Device:C") (at 88 117.62 0) (unit 1)
+    (in_bom yes) (on_board yes) (dnp no)
+      (property "Reference" "C5b" (at 90.54 115.08 0)
+        (effects (font (size 1.27 1.27))))
+      (property "Value" "10nF X7R 0603 (VDD HF²)" (at 90.54 118.89 0)
+        (effects (font (size 1.27 1.27))))
+      (property "Footprint" "Capacitor_SMD:C_0603_1608Metric" (at 88 117.62 0)
+        (effects (font (size 1.27 1.27)) hide))
+      (property "Datasheet" "~" (at 88 117.62 0)
+        (effects (font (size 1.27 1.27)) hide))
+      (property "MPN" "0603B103K500NT" (at 90.54 121.43 0)
+        (effects (font (size 1.27 1.27)) hide))
+      (property "LCSC" "C57112" (at 90.54 122.7 0)
         (effects (font (size 1.27 1.27)) hide))
     (instances
       (project "field_ambience"
         (path "/ae4d8abd-ab57-48bd-a18a-f37b38917ad2" (reference "C5b") (unit 1)))))
-  (symbol (lib_id "Power:GND") (at 103 123.81 270) (unit 1)
-    (in_bom yes) (on_board yes) (dnp no)
-      (property "Reference" "#PWR_C5b" (at 105.54 121.27 0)
-        (effects (font (size 1.27 1.27))))
-      (property "Value" "GND" (at 105.54 125.08 0)
-        (effects (font (size 1.27 1.27))))
-      (property "Footprint" "" (at 103 123.81 0)
-        (effects (font (size 1.27 1.27)) hide))
-      (property "Datasheet" "~" (at 103 123.81 0)
+  (symbol (lib_id "Power:GND") (at 88 123.81 270) (unit 1)
+    (in_bom yes) (on_board yes) (dnp no)
+      (property "Reference" "#PWR_C5b" (at 90.54 121.27 0)
+        (effects (font (size 1.27 1.27))))
+      (property "Value" "GND" (at 90.54 125.08 0)
+        (effects (font (size 1.27 1.27))))
+      (property "Footprint" "" (at 88 123.81 0)
+        (effects (font (size 1.27 1.27)) hide))
+      (property "Datasheet" "~" (at 88 123.81 0)
         (effects (font (size 1.27 1.27)) hide))
     (instances
@@
       (property "Datasheet" "~" (at 158 153.49 0)
         (effects (font (size 1.27 1.27)) hide))
-      (property "MPN" "CL21A106KOQNNNG-class" (at 160.54 157.3 0)
+      (property "MPN" "CL21A106KAYNNNE" (at 160.54 157.3 0)
         (effects (font (size 1.27 1.27)) hide))
       (property "LCSC" "C15850" (at 160.54 158.57000000000002 0)
@@
       (property "Datasheet" "~" (at 164 153.49 0)
         (effects (font (size 1.27 1.27)) hide))
-      (property "MPN" "CL10B104KO8NNNC-class" (at 166.54 157.3 0)
+      (property "MPN" "CC0603KRX7R9BB104" (at 166.54 157.3 0)
         (effects (font (size 1.27 1.27)) hide))
       (property "LCSC" "C14663" (at 166.54 158.57000000000002 0)
@@
       (property "Datasheet" "~" (at 327.7 108.49 0)
         (effects (font (size 1.27 1.27)) hide))
-      (property "MPN" "CL21A106KOQNNNG-class" (at 330.24 112.3 0)
+      (property "MPN" "CL21A106KAYNNNE" (at 330.24 112.3 0)
         (effects (font (size 1.27 1.27)) hide))
       (property "LCSC" "C15850" (at 330.24 113.57 0)
@@
       (property "Datasheet" "~" (at 333.7 108.49 0)
         (effects (font (size 1.27 1.27)) hide))
-      (property "MPN" "CL10B104KO8NNNC-class" (at 336.24 112.3 0)
+      (property "MPN" "CC0603KRX7R9BB104" (at 336.24 112.3 0)
         (effects (font (size 1.27 1.27)) hide))
       (property "LCSC" "C14663" (at 336.24 113.57 0)
@@
     (stroke (width 0) (type default))
 )
-  (wire (pts (xy 108 113.81) (xy 113 113.81))
-    (stroke (width 0) (type default))
-)
-  (wire (pts (xy 108 121.43) (xy 108 123.81))
-    (stroke (width 0) (type default))
-)
-  (wire (pts (xy 103 113.81) (xy 108 113.81))
-    (stroke (width 0) (type default))
-)
-  (wire (pts (xy 103 121.43) (xy 103 123.81))
+  (wire (pts (xy 88 113.81) (xy 113 113.81))
+    (stroke (width 0) (type default))
+)
+  (wire (pts (xy 93 121.43) (xy 93 123.81))
+    (stroke (width 0) (type default))
+)
+  (wire (pts (xy 88 121.43) (xy 88 123.81))
     (stroke (width 0) (type default))
 )
@@
   (junction (at 113 113.81) (diameter 0) (color 0 0 0 0)
 )
-  (junction (at 108 113.81) (diameter 0) (color 0 0 0 0)
+  (junction (at 93 113.81) (diameter 0) (color 0 0 0 0)
 )
   (junction (at 113 121.42999999999999) (diameter 0) (color 0 0 0 0)
+)
+  (junction (at 104 113.81) (diameter 0) (color 0 0 0 0)
 )
   (junction (at 113 123.97) (diameter 0) (color 0 0 0 0)
@@
     (effects (font (size 1.524 1.524)) (justify right))
 )
+  (no_connect (at 312.7 136.51)
+)
+  (no_connect (at 312.7 133.97)
+)
+  (no_connect (at 312.7 131.43)
+)
+  (no_connect (at 312.7 128.89)
+)
+  (no_connect (at 312.7 126.35)
+)
+  (no_connect (at 312.7 123.81)
+)
+  (no_connect (at 312.7 121.27)
+)
+  (no_connect (at 312.7 118.72999999999999)
+)
   (sheet_instances
