File: field-ambience-current/kicad/pico.kicad_sch (KiCad schematic)
At the start: 10 parts, among them J4 SWD 1.27mm (SWCLK/GND/SWDIO), SW11 Reset 6mm SMD, SW12 BOOTSEL 6mm SMD (DNP for THT-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, U1 Raspberry_Pi_Pico2 (RP2350)

Commit message: pcb(bom): r12-B12 — 9 falsche LCSC-Codes via jlcsearch-Audit korrigiert + r12-B11 TPS-Package-Blocker
JLC-Pricing-Estimate-Run hat 9 falsche LCSC-Codes im Generator aufgedeckt.
Alle MPN-Strings waren korrekt, aber die zugewiesenen LCSC-Codes pointed
auf völlig andere Teile. Bei sofortiger JLC-Bestellung wäre der Prototyp
DOA gewesen (BAT_SENSE-Divider 130Ω/130Ω statt 100k/100k, Boost-FB 15Ω/0.21k
statt 200k/39k, alle LEDs nicht-existent, etc.).

Korrigierte Mappings (via jlcsearch-API-Verifikation):
- 100kΩ 0603 (R_BAT_DIV_TOP/BOT, R_VBUS_PD): C22796 → C25803 (Basic)
- 200kΩ 0603 (R23): C22810 → C25811 (Basic)
- 39kΩ 0603 (R24): C25090 → C23153 (Basic)
- 390Ω 0603 (R_LED6-15, R_LED_STATUS): C23289 → C23151 (Basic)
- MCP73831T-2ACI/OT (U7): C14879 → C424093 (Extended)
- DMG2305UX-7 (Q1): C147074 → C150470 (Extended)
- SWPA6045S2R2MT (L1): C32330 → C83455 (Extended)
- S2B-PH-SM4-TB SMD (J9): C146061 → C295747 (Extended)
- 0603 white LED (LED1, LED6-15): C72043 → C965808 XL-1608UWC-04 (Extended)

Neuer BLOCKER r12-B11: TPS61089-Package-Mismatch
SPEC §2.2 spezifiziert TPS61089RNSR (QFN-12 3×3mm), aber LCSC hat nur
TPS61089RNRR (VQFN-11 2×2.5mm HotRod, anderer Footprint + Pinout).
Generator markiert LCSC vorerst als "TBD-USER-SUPPLY-or-RNRR-refactor"
bis User-Decision. 3 Lösungswege in PCB_TODO r12-B11 dokumentiert
(RNRR-Refactor / RNSR-Konsignierung / Hand-Solder).

Side-Effekt: 4 der korrigierten Resistor-SKUs sind Basic (kein Extended-
Setup-Fee) → spart $12 bei 5-Boards. Extended-SKU-Count 23 → 19.

JLC-Cost-Estimate aktualisiert in CHANGELOG: 5 Prototyp-Boards ~$567
(JLC $294 + User-Supplied $272 + Battery/OLED/Choc/Pico/Speaker), per
Board ~$113. Bei 100 Stück ~$6884 (~$69/Board).

Generator/SPEC/PCB_TODO/CHANGELOG synchron. Analyzer-Status unverändert
(LCSC sind Metadata, keine Connectivity-Änderung).

https://claude.ai/code/session_01K5kLTFpDCCoYwx2dq6RkAv
Parts:
- R_BAT_DIV_BOT, R_BAT_DIV_TOP: LCSC C22796 -> C25803
Changed lines of the file:
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@@
       (property "MPN" "0603WAF1003T5E" (at 137.54 102.54 0)
         (effects (font (size 1.27 1.27)) hide))
-      (property "LCSC" "C22796" (at 137.54 103.81 0)
+      (property "LCSC" "C25803" (at 137.54 103.81 0)
         (effects (font (size 1.27 1.27)) hide))
     (instances
@@
       (property "MPN" "0603WAF1003T5E" (at 132.54 112.54 0)
         (effects (font (size 1.27 1.27)) hide))
-      (property "LCSC" "C22796" (at 132.54 113.81 0)
+      (property "LCSC" "C25803" (at 132.54 113.81 0)
         (effects (font (size 1.27 1.27)) hide))
     (instances
