File: field-ambience-current/kicad/encoder.kicad_sch (KiCad schematic)
At the start: 24 parts

Commit message: fix(bom): make entire BOM correctly JLC-orderable — 7 real part errors fixed
Verified every LCSC number against jlcsearch for existence, stock, AND that
it resolves to the intended value/package. Found 7 parts that would have
built WRONG or were unorderable:

CRITICAL value/package errors (LCSC pointed at the wrong part):
- R_VOL_L/R: C25092 = 22ohm 0402  -> C4184  (real 20k 0603, Basic).
  Was wrong value AND footprint; would have wrecked the PAM8403 input gain.
- R_LO_L/R:  C22962 = 220ohm       -> C23345 (real 22ohm 0603, Basic).
- R_BCK/LRCK/DOUT: C23138 = 330ohm -> C23140 (real 33ohm 0603, Basic).

Unorderable -> assigned real in-stock parts:
- J8 jack:  C2884109 (nonexistent) -> C431535 (PJ-320D SMD).
- C_BULK:   placeholder            -> C46550395 (1000uF 16V SMD D10x10.5).
- LED1:     no LCSC                -> C965818 (white 0805).
- R1:       C22548 Extended        -> C21190 Basic (prior commit).

Also aligned all MPN text to the actual LCSC part (Yageo text vs Uni Royal/
Samsung parts JLC ships) so the BOM is internally consistent.

Re-verified: 25 distinct LCSC, all in stock, ZERO value/package mismatches,
14 Basic / 11 Extended. SPEC §4 stale refs (C_BULK/J8/R_LO) updated.
MEINE_TODO Abschnitt 0 rewritten with the full orderability result.

Self-supply parts (Pico, OLED, speakers, Choc sockets, EC11, headers) keep
no LCSC by design — JLC cannot assemble those.

https://claude.ai/code/session_01K5kLTFpDCCoYwx2dq6RkAv
Parts:
- R10, R11, R12, R13, R14, R15, R16, R17, R18, R7, R8, R9: MPN RC0603FR-0710KL -> 0603WAF1002T5E
Changed lines of the file:
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@@
       (property "Datasheet" "~" (at 128 61.11 0)
         (effects (font (size 1.27 1.27)) hide))
-      (property "MPN" "RC0603FR-0710KL" (at 130.54 64.92 0)
+      (property "MPN" "0603WAF1002T5E" (at 130.54 64.92 0)
         (effects (font (size 1.27 1.27)) hide))
       (property "LCSC" "C25804" (at 130.54 66.19 0)
@@
       (property "Datasheet" "~" (at 132 66.19 0)
         (effects (font (size 1.27 1.27)) hide))
-      (property "MPN" "RC0603FR-0710KL" (at 134.54 70.0 0)
+      (property "MPN" "0603WAF1002T5E" (at 134.54 70.0 0)
         (effects (font (size 1.27 1.27)) hide))
       (property "LCSC" "C25804" (at 134.54 71.27 0)
@@
       (property "Datasheet" "~" (at 152 63.64999999999999 0)
         (effects (font (size 1.27 1.27)) hide))
-      (property "MPN" "RC0603FR-0710KL" (at 154.54 67.46 0)
+      (property "MPN" "0603WAF1002T5E" (at 154.54 67.46 0)
         (effects (font (size 1.27 1.27)) hide))
       (property "LCSC" "C25804" (at 154.54 68.72999999999999 0)
@@
       (property "Datasheet" "~" (at 128 96.11 0)
         (effects (font (size 1.27 1.27)) hide))
-      (property "MPN" "RC0603FR-0710KL" (at 130.54 99.92 0)
+      (property "MPN" "0603WAF1002T5E" (at 130.54 99.92 0)
         (effects (font (size 1.27 1.27)) hide))
       (property "LCSC" "C25804" (at 130.54 101.19 0)
@@
       (property "Datasheet" "~" (at 132 101.19 0)
         (effects (font (size 1.27 1.27)) hide))
-      (property "MPN" "RC0603FR-0710KL" (at 134.54 105.0 0)
+      (property "MPN" "0603WAF1002T5E" (at 134.54 105.0 0)
         (effects (font (size 1.27 1.27)) hide))
       (property "LCSC" "C25804" (at 134.54 106.27 0)
@@
       (property "Datasheet" "~" (at 152 98.64999999999999 0)
         (effects (font (size 1.27 1.27)) hide))
-      (property "MPN" "RC0603FR-0710KL" (at 154.54 102.46 0)
+      (property "MPN" "0603WAF1002T5E" (at 154.54 102.46 0)
         (effects (font (size 1.27 1.27)) hide))
       (property "LCSC" "C25804" (at 154.54 103.72999999999999 0)
@@
       (property "Datasheet" "~" (at 128 131.10999999999999 0)
         (effects (font (size 1.27 1.27)) hide))
-      (property "MPN" "RC0603FR-0710KL" (at 130.54 134.92 0)
+      (property "MPN" "0603WAF1002T5E" (at 130.54 134.92 0)
         (effects (font (size 1.27 1.27)) hide))
       (property "LCSC" "C25804" (at 130.54 136.19 0)
@@
       (property "Datasheet" "~" (at 132 136.19 0)
         (effects (font (size 1.27 1.27)) hide))
-      (property "MPN" "RC0603FR-0710KL" (at 134.54 140.0 0)
+      (property "MPN" "0603WAF1002T5E" (at 134.54 140.0 0)
         (effects (font (size 1.27 1.27)) hide))
       (property "LCSC" "C25804" (at 134.54 141.27 0)
@@
       (property "Datasheet" "~" (at 152 133.65 0)
         (effects (font (size 1.27 1.27)) hide))
-      (property "MPN" "RC0603FR-0710KL" (at 154.54 137.46 0)
+      (property "MPN" "0603WAF1002T5E" (at 154.54 137.46 0)
         (effects (font (size 1.27 1.27)) hide))
       (property "LCSC" "C25804" (at 154.54 138.73000000000002 0)
@@
       (property "Datasheet" "~" (at 128 166.10999999999999 0)
         (effects (font (size 1.27 1.27)) hide))
-      (property "MPN" "RC0603FR-0710KL" (at 130.54 169.92 0)
+      (property "MPN" "0603WAF1002T5E" (at 130.54 169.92 0)
         (effects (font (size 1.27 1.27)) hide))
       (property "LCSC" "C25804" (at 130.54 171.19 0)
@@
       (property "Datasheet" "~" (at 132 171.19 0)
         (effects (font (size 1.27 1.27)) hide))
-      (property "MPN" "RC0603FR-0710KL" (at 134.54 175.0 0)
+      (property "MPN" "0603WAF1002T5E" (at 134.54 175.0 0)
         (effects (font (size 1.27 1.27)) hide))
       (property "LCSC" "C25804" (at 134.54 176.27 0)
@@
       (property "Datasheet" "~" (at 152 168.65 0)
         (effects (font (size 1.27 1.27)) hide))
-      (property "MPN" "RC0603FR-0710KL" (at 154.54 172.46 0)
+      (property "MPN" "0603WAF1002T5E" (at 154.54 172.46 0)
         (effects (font (size 1.27 1.27)) hide))
       (property "LCSC" "C25804" (at 154.54 173.73000000000002 0)

Commit message: pcb(r18.5): Schematic-Migration Phase 3 — STM32H743 + LCD im Generator, Repo-Audit-Fixes
KERN: generate_kicad_project.py erzeugt jetzt die H7-Architektur.

NEU stm32h743.kicad_sch (ersetzt pico.kicad_sch -> kicad/legacy_pico2/):
- 100-Pin-Symbol 1:1 aus offizieller KiCad-Lib (MCU_ST_STM32H7),
  doppelt verifiziert gegen SPEC v0.7 §5 / DS12110 Rev 5 Table 8 —
  alle 52 belegten Zuordnungen identisch (zwei unabhängige Quellen)
- alle SPEC-§5-Netze verdrahtet, 48 Reserve-GPIOs no_connect
- Support: HSE Y1 ABLS-8.000MHZ-B4-T (C596838) + 2x22pF, VCAP 2x2.2uF
  (DS12110 Tab.24), 5x(4.7uF+100nF) VDD-Bank, VDDA-Ferrit C84094 +
  1uF+100nF, BOOT0-PD 10k, NRST-PU 10k+100nF, SWD-J4 (PA13/PA14/GND),
  BAT-Teiler 100k/100k+10nF an PA3, Status-LED PD8, USB-FS PA11/PA12
  (USBLC6-ESD bleibt davor), MIDI_TX-Netz (PD5)

NEU lcd.kicad_sch (ersetzt oled.kicad_sch -> legacy): 8-Pin-ST7789
per SPEC §6 + C6b/C6c + Backlight: PCA9685-Kanal-12 -> LCD_BLK_PWM ->
2N7002 Low-Side + 100k-PD. Netze OLED_* -> LCD_*.

power_tree: U5 AP7361A-33 LDO (+5V->+3V3) + Cin 1uF/Cout 2.2uF +
EN->IN. Pico-SMPS entfällt. PICO_USB_* -> USB_DM/USB_DP.

mcp: GPB5 = VOL_SW (SPEC §5.4 — lag bis r17 entgegen der SPEC am
Pico-GPIO), PCA-Kanal 12 = LCD_BLK_PWM. Root-Brücken umgebaut,
kicad_pro-Sheetliste: Battery ergänzt (fehlte).

AUDIT-FINDINGS (verifiziert, nicht aus dem Alt-Audit übernommen):
- F-6 NEU 🔴: SPEC-§4-U5-LCSC C156144 ist ein 910R-WIDERSTAND
  (LCSC-Web verifiziert) — hätte bei JLC einen R als LDO bestückt.
  SPEC korrigiert (Kandidat C150719), Symbol trägt TBD-VERIFY.
- B-LDO 🔴: AP7361A-SOT-89-5-Pinout-Annahme (1=ADJ/NC,2=OUT,3=IN,
  4=GND,5=EN aus AP7361-DS33626-Lesart; A-Datasheet war HTTP 403) —
  als PIN_VERIFY am Symbol + PCB_LAYOUT_STATUS dokumentiert.
- B-SW12 🔴: SW6-10 (HX 12x12) auf ~6mm-TL3342-Pattern — als
  FP_MISMATCH-Property an allen 5 Symbolen markiert.
- F-2-Teilfix: Encoder-MPN -> EC11J1525402, Bourns-PEC11R-PDF nach
  datasheets/legacy/ (falsches Teil); ALPS-Drawing offen.
- F-1: T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
Parts:
- EN1, EN2, EN3, EN4: LCSC TBD (mehrere EC11-Varianten verfügbar) -> EC11J1525402 (ALPSALPINE, SPEC §4) — F-2: LCSC + Land-Patte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
Changed lines of the file:
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@@
       (property "Footprint" "Rotary_Encoder:RotaryEncoder_Alps_EC11E-Switch_Vertical_H20mm" (at 140.0 70 0)
         (effects (font (size 1.27 1.27)) hide))
-      (property "Datasheet" "https://www.bourns.com/docs/Product-Datasheets/PEC11R.pdf" (at 140.0 70 0)
+      (property "Datasheet" "TODO-F2: ALPS EC11J1525402 Drawing beschaffen (Bourns-PEC11R-PDF war falsches Teil)" (at 140.0 70 0)
         (effects (font (size 1.27 1.27)) hide))
       (property "MPN" "PEC11R-4215F-S0024" (at 142.54 73.81 0)
         (effects (font (size 1.27 1.27)) hide))
-      (property "LCSC" "TBD (mehrere EC11-Varianten verfügbar)" (at 142.54 75.08 0)
+      (property "LCSC" "EC11J1525402 (ALPSALPINE, SPEC §4) — F-2: LCSC + Land-Pattern-Verify offen" (at 142.54 75.08 0)
         (effects (font (size 1.27 1.27)) hide))
     (instances
@@
       (property "Footprint" "Rotary_Encoder:RotaryEncoder_Alps_EC11E-Switch_Vertical_H20mm" (at 140.0 105 0)
         (effects (font (size 1.27 1.27)) hide))
-      (property "Datasheet" "https://www.bourns.com/docs/Product-Datasheets/PEC11R.pdf" (at 140.0 105 0)
+      (property "Datasheet" "TODO-F2: ALPS EC11J1525402 Drawing beschaffen (Bourns-PEC11R-PDF war falsches Teil)" (at 140.0 105 0)
         (effects (font (size 1.27 1.27)) hide))
       (property "MPN" "PEC11R-4215F-S0024" (at 142.54 108.81 0)
         (effects (font (size 1.27 1.27)) hide))
-      (property "LCSC" "TBD (mehrere EC11-Varianten verfügbar)" (at 142.54 110.08 0)
+      (property "LCSC" "EC11J1525402 (ALPSALPINE, SPEC §4) — F-2: LCSC + Land-Pattern-Verify offen" (at 142.54 110.08 0)
         (effects (font (size 1.27 1.27)) hide))
     (instances
@@
       (property "Footprint" "Rotary_Encoder:RotaryEncoder_Alps_EC11E-Switch_Vertical_H20mm" (at 140.0 140 0)
         (effects (font (size 1.27 1.27)) hide))
-      (property "Datasheet" "https://www.bourns.com/docs/Product-Datasheets/PEC11R.pdf" (at 140.0 140 0)
+      (property "Datasheet" "TODO-F2: ALPS EC11J1525402 Drawing beschaffen (Bourns-PEC11R-PDF war falsches Teil)" (at 140.0 140 0)
         (effects (font (size 1.27 1.27)) hide))
       (property "MPN" "PEC11R-4215F-S0024" (at 142.54 143.81 0)
         (effects (font (size 1.27 1.27)) hide))
-      (property "LCSC" "TBD (mehrere EC11-Varianten verfügbar)" (at 142.54 145.08 0)
+      (property "LCSC" "EC11J1525402 (ALPSALPINE, SPEC §4) — F-2: LCSC + Land-Pattern-Verify offen" (at 142.54 145.08 0)
         (effects (font (size 1.27 1.27)) hide))
     (instances
@@
       (property "Footprint" "Rotary_Encoder:RotaryEncoder_Alps_EC11E-Switch_Vertical_H20mm" (at 140.0 175 0)
         (effects (font (size 1.27 1.27)) hide))
-      (property "Datasheet" "https://www.bourns.com/docs/Product-Datasheets/PEC11R.pdf" (at 140.0 175 0)
+      (property "Datasheet" "TODO-F2: ALPS EC11J1525402 Drawing beschaffen (Bourns-PEC11R-PDF war falsches Teil)" (at 140.0 175 0)
         (effects (font (size 1.27 1.27)) hide))
       (property "MPN" "PEC11R-4215F-S0024" (at 142.54 178.81 0)
         (effects (font (size 1.27 1.27)) hide))
-      (property "LCSC" "TBD (mehrere EC11-Varianten verfügbar)" (at 142.54 180.08 0)
-        (effects (font (size 1.27 1.27)) hide))
-    (instances
+      (property "LCSC" "EC11J1525402 (ALPSALPINE, SPEC §4) — F-2: LCSC + Land-Pattern-Verify offen" (at 142.54 180.08 0)
+        (effects (font (size 1.27 1.27)) hide))
+    (instances

Commit message: pcb(r18.6): Engineering-Verifikation — AP7361C-Pinout-Fix, TPS61089-Quelle, Custom-FP, BOM-LCSC, ADR-MIDI
Reaktion auf User-Korrekturen aus öffentlichen Datasheets. Vier
🔴-Blocker geschlossen, einer auf eine Design-Entscheidung umklassifiziert.

=== AP7361A-Pinout war FALSCH — gefixt + AP7361C ===

r18.5-Annahme: 1=ADJ/NC, 2=OUT, 3=IN, 4=GND, 5=EN.
Korrekt (Diodes-DS via mouser.de/datasheet/3/175/1/AP7361.pdf,
User-verifiziert):
    1=EN, 2=GND, 3=ADJ/NC, 4=IN, 5=OUT

Hätte zu einem totem Board geführt (IN/OUT/EN vertauscht).

Zusätzlich:
- Symbol auf AP7361C umbenannt (Diodes markiert AP7361 als NRND ->
  use AP7361C; gleicher SOT-89-5-Pinout)
- AP7361C-33Y5-13 = LCSC C460397 (SOT-89-5) statt r18.5-Kandidat
  C150719 (= SOT-223, falsches Package; verworfen)
- Cin/Cout 4.7 µF X5R 0603 (DS-Empfehlung, statt 1µF/2.2µF)
- Symbol-Pinmap + power_tree-Verdrahtung umgebaut: EN-Pin liegt
  jetzt links oben (statt links unten), IN links unten, OUT
  rechts oben — neu gerechnete Stub-Wires + Junctions

=== TPS61089-Footprint + Datenblatt-Anchor ===

- Symbol-Pinmap (1=FSW … 11=SW) verifiziert gegen TI Rev C Tabelle 6-1
  (User-Quelle ti.com/lit/gpn/tps61089) — als PIN_SOURCE-Property
- Footprint-Name auf RNR0011A-Konvention 2.0x2.5mm VQFN-HR
- RNSR-PDF → datasheets/legacy/TPS61089RNSR_wrong_variant.pdf

=== Encoder C209762 (NRND, Prototype-OK) ===

- MPN EC11J1525402, LCSC C209762 (JLCPCB-verifiziert)
- Datasheet-Link auf JLCPCB-Detail-Seite (ALPS-Drawing nicht öffentlich)
- Status: NRND als Property — Prototype-OK, Serie braucht Ersatztyp
- FP_VERIFY-Hinweis (EC11J ist SMD, der KiCad-Standard-FP EC11E ist THT)

=== Custom-Footprint für HX 12x12 (SW6-10) ===

- libraries/field_ambience.pretty/SW_HX_12x12x7.3_SMD-4P.kicad_mod
  basierend auf LCSC-Daten von C36498966:
  - SMD-4P, 11.8x11.8mm Body, 7.3mm Höhe
  - 4 Pads je 2.5x1.5mm auf 7mm-Pitch (X+Y)
  - SPST: gegenüberliegende Pads verbunden (1↔1, 2↔2)
  - Silkscreen + Pin-1-Dot + Courtyard +0.25mm IPC-7351B
- fp-lib-table um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
Parts:
- EN1, EN2, EN3, EN4: FP_VERIFY (none) -> F-2: KiCad-Standard-FP ist EC11E (THT-Stems); EC11J ist SMD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; LCSC EC11J1525402 (ALPSALPINE, SPEC §4) — F-2: LCSC + Land-Patte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 -> C209762; MPN PEC11R-4215F-S0024 -> EC11J1525402; Manufacturer (none) -> ALPSALPINE; Package (none) -> SMD, 15 pulses / 30 detents, push switch; Status (none) -> NRND (ALPS marks as Not Recommended For New Designs) — Prot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
Changed lines of the file:
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@@
       (property "Footprint" "Rotary_Encoder:RotaryEncoder_Alps_EC11E-Switch_Vertical_H20mm" (at 140.0 70 0)
         (effects (font (size 1.27 1.27)) hide))
-      (property "Datasheet" "TODO-F2: ALPS EC11J1525402 Drawing beschaffen (Bourns-PEC11R-PDF war falsches Teil)" (at 140.0 70 0)
-        (effects (font (size 1.27 1.27)) hide))
-      (property "MPN" "PEC11R-4215F-S0024" (at 142.54 73.81 0)
-        (effects (font (size 1.27 1.27)) hide))
-      (property "LCSC" "EC11J1525402 (ALPSALPINE, SPEC §4) — F-2: LCSC + Land-Pattern-Verify offen" (at 142.54 75.08 0)
+      (property "Datasheet" "https://jlcpcb.com/partdetail/C209762" (at 140.0 70 0)
+        (effects (font (size 1.27 1.27)) hide))
+      (property "MPN" "EC11J1525402" (at 142.54 73.81 0)
+        (effects (font (size 1.27 1.27)) hide))
+      (property "Manufacturer" "ALPSALPINE" (at 142.54 75.08 0)
+        (effects (font (size 1.27 1.27)) hide))
+      (property "LCSC" "C209762" (at 142.54 76.35 0)
+        (effects (font (size 1.27 1.27)) hide))
+      (property "Package" "SMD, 15 pulses / 30 detents, push switch" (at 142.54 77.62 0)
+        (effects (font (size 1.27 1.27)) hide))
+      (property "Status" "NRND (ALPS marks as Not Recommended For New Designs) — Prototype-OK, Serie: Ersatztyp wählen" (at 142.54 78.89 0)
+        (effects (font (size 1.27 1.27)) hide))
+      (property "FP_VERIFY" "F-2: KiCad-Standard-FP ist EC11E (THT-Stems); EC11J ist SMD-Bauform. Vor Layout Land-Pattern gegen JLCPCB-EasyEDA-Drawing für C209762 abgleichen oder eigenen FP zeichnen." (at 142.54 80.16 0)
         (effects (font (size 1.27 1.27)) hide))
     (instances
@@
       (property "Footprint" "Rotary_Encoder:RotaryEncoder_Alps_EC11E-Switch_Vertical_H20mm" (at 140.0 105 0)
         (effects (font (size 1.27 1.27)) hide))
-      (property "Datasheet" "TODO-F2: ALPS EC11J1525402 Drawing beschaffen (Bourns-PEC11R-PDF war falsches Teil)" (at 140.0 105 0)
-        (effects (font (size 1.27 1.27)) hide))
-      (property "MPN" "PEC11R-4215F-S0024" (at 142.54 108.81 0)
-        (effects (font (size 1.27 1.27)) hide))
-      (property "LCSC" "EC11J1525402 (ALPSALPINE, SPEC §4) — F-2: LCSC + Land-Pattern-Verify offen" (at 142.54 110.08 0)
+      (property "Datasheet" "https://jlcpcb.com/partdetail/C209762" (at 140.0 105 0)
+        (effects (font (size 1.27 1.27)) hide))
+      (property "MPN" "EC11J1525402" (at 142.54 108.81 0)
+        (effects (font (size 1.27 1.27)) hide))
+      (property "Manufacturer" "ALPSALPINE" (at 142.54 110.08 0)
+        (effects (font (size 1.27 1.27)) hide))
+      (property "LCSC" "C209762" (at 142.54 111.35 0)
+        (effects (font (size 1.27 1.27)) hide))
+      (property "Package" "SMD, 15 pulses / 30 detents, push switch" (at 142.54 112.62 0)
+        (effects (font (size 1.27 1.27)) hide))
+      (property "Status" "NRND (ALPS marks as Not Recommended For New Designs) — Prototype-OK, Serie: Ersatztyp wählen" (at 142.54 113.89 0)
+        (effects (font (size 1.27 1.27)) hide))
+      (property "FP_VERIFY" "F-2: KiCad-Standard-FP ist EC11E (THT-Stems); EC11J ist SMD-Bauform. Vor Layout Land-Pattern gegen JLCPCB-EasyEDA-Drawing für C209762 abgleichen oder eigenen FP zeichnen." (at 142.54 115.16 0)
         (effects (font (size 1.27 1.27)) hide))
     (instances
@@
       (property "Footprint" "Rotary_Encoder:RotaryEncoder_Alps_EC11E-Switch_Vertical_H20mm" (at 140.0 140 0)
         (effects (font (size 1.27 1.27)) hide))
-      (property "Datasheet" "TODO-F2: ALPS EC11J1525402 Drawing beschaffen (Bourns-PEC11R-PDF war falsches Teil)" (at 140.0 140 0)
-        (effects (font (size 1.27 1.27)) hide))
-      (property "MPN" "PEC11R-4215F-S0024" (at 142.54 143.81 0)
-        (effects (font (size 1.27 1.27)) hide))
-      (property "LCSC" "EC11J1525402 (ALPSALPINE, SPEC §4) — F-2: LCSC + Land-Pattern-Verify offen" (at 142.54 145.08 0)
+      (property "Datasheet" "https://jlcpcb.com/partdetail/C209762" (at 140.0 140 0)
+        (effects (font (size 1.27 1.27)) hide))
+      (property "MPN" "EC11J1525402" (at 142.54 143.81 0)
+        (effects (font (size 1.27 1.27)) hide))
+      (property "Manufacturer" "ALPSALPINE" (at 142.54 145.08 0)
+        (effects (font (size 1.27 1.27)) hide))
+      (property "LCSC" "C209762" (at 142.54 146.35 0)
+        (effects (font (size 1.27 1.27)) hide))
+      (property "Package" "SMD, 15 pulses / 30 detents, push switch" (at 142.54 147.62 0)
+        (effects (font (size 1.27 1.27)) hide))
+      (property "Status" "NRND (ALPS marks as Not Recommended For New Designs) — Prototype-OK, Serie: Ersatztyp wählen" (at 142.54 148.89 0)
+        (effects (font (size 1.27 1.27)) hide))
+      (property "FP_VERIFY" "F-2: KiCad-Standard-FP ist EC11E (THT-Stems); EC11J ist SMD-Bauform. Vor Layout Land-Pattern gegen JLCPCB-EasyEDA-Drawing für C209762 abgleichen oder eigenen FP zeichnen." (at 142.54 150.16 0)
         (effects (font (size 1.27 1.27)) hide))
     (instances
@@
       (property "Footprint" "Rotary_Encoder:RotaryEncoder_Alps_EC11E-Switch_Vertical_H20mm" (at 140.0 175 0)
         (effects (font (size 1.27 1.27)) hide))
-      (property "Datasheet" "TODO-F2: ALPS EC11J1525402 Drawing beschaffen (Bourns-PEC11R-PDF war falsches Teil)" (at 140.0 175 0)
-        (effects (font (size 1.27 1.27)) hide))
-      (property "MPN" "PEC11R-4215F-S0024" (at 142.54 178.81 0)
-        (effects (font (size 1.27 1.27)) hide))
-      (property "LCSC" "EC11J1525402 (ALPSALPINE, SPEC §4) — F-2: LCSC + Land-Pattern-Verify offen" (at 142.54 180.08 0)
-        (effects (font (size 1.27 1.27)) hide))
-    (instances
+      (property "Datasheet" "https://jlcpcb.com/partdetail/C209762" (at 140.0 175 0)
+        (effects (font (size 1.27 1.27)) hide))
+      (property "MPN" "EC11J1525402" (at 142.54 178.81 0)
+        (effects (font (size 1.27 1.27)) hide))
+      (property "Manufacturer" "ALPSALPINE" (at 142.54 180.08 0)
+        (effects (font (size 1.27 1.27)) hide))
+      (property "LCSC" "C209762" (at 142.54 181.35 0)
+        (effects (font (size 1.27 1.27)) hide))
+      (property "Package" "SMD, 15 pulses / 30 detents, push switch" (at 142.54 182.62 0)
+        (effects (font (size 1.27 1.27)) hide))
+      (property "Status" "NRND (ALPS marks as Not Recommended For New Designs) — Prototype-OK, Serie: Ersatztyp wählen" (at 142.54 183.89 0)
+        (effects (font (size 1.27 1.27)) hide))
+      (property "FP_VERIFY" "F-2: KiCad-Standard-FP ist EC11E (THT-Stems); EC11J ist SMD-Bauform. Vor Layout Land-Pattern gegen JLCPCB-EasyEDA-Drawing für C209762 abgleichen oder eigenen FP zeichnen." (at 142.54 185.16 0)
+        (effects (font (size 1.27 1.27)) hide))
+    (instances
