File: field-ambience-current/kicad/encoder.kicad_sch (KiCad schematic)
At the start: 24 parts

Commit message: pcb(r18.12): Pre-Layout-Cleanup — Polymer-Bulk-Cap + EC11J Custom-Draft-FP
Zwei offene Pre-Layout-Punkte adressiert.

=== C_BULK Polymer-Wechsel (loest ADR-0011 Konflikt) ===

1000uF Alu-Elko (10.5mm Hoehe — passte nicht in 8mm-Top-Zone) ersetzt durch:
- C_BULK: 470uF 16V Polymer in EIA-7343-31 (D-Case, ~2mm Hoehe, ESR<15mOhm)
- C_BULK2: 220uF 10V X5R MLCC 1210 parallel

Effektive Bulk-Kapazitaet ~690uF, aber ESR ~10mOhm statt ~25mOhm beim Alu.
Class-D-Bass-Transienten sauberer (ADR-0010 Punkt 4 Anti-Kratzig-Hebel
verstaerkt). Title-Block-Comment synchronisiert.

LCSC-Nummern noch TBD-VERIFY: Panasonic SVPF / Kemet T520D fuer Polymer;
CL32A227KQVNNNE-Klasse fuer 220uF MLCC. Vor BOM-Freeze final pruefen.

=== EC11J Custom-Footprint (FP_VERIFY letzter Punkt) ===

libraries/field_ambience.pretty/RotaryEncoder_ALPS_EC11J_SMD.kicad_mod NEU:
- aus dokumentierten ALPS-EC11J-Standard-Maßen (12x13.4mm Body, 20mm Schaft)
- 5 SMD-Pads + 2 Mounting-Tabs
- Pad-Pitch 2.5mm, Pad 1.4x1.4mm, Mounting-Tabs 1.8x3mm bei +-6mm
- Status FP_DRAFT (nicht FP_NOTE) — vor Fab gegen EasyEDA-Export von
  C209762 verifizieren (Property im Schematic markiert)

4 Encoder-Instanzen referenzieren jetzt den Custom-FP statt des KiCad-
Standard-EC11E-THT-FP (der ohnehin nicht zur SMD-Bauform passte).

=== Validierung ===

paren 8/8 PASS - Crossref 7/7 PASS - 4 Encoder-Instanzen mit neuem FP,
0 EC11E-Reste - Polymer + MLCC parallel sauber im power_tree platziert -
Title-Block-stale-Kommentar gefixt.

=== Scores ===

- Footprint-Verifikation 8 -> 9 (EC11J Draft-FP geschlossen)
- Mechanical / Enclosure 4 -> 5 (C_BULK-Konflikt aufgeloest)
- BOM-Sourcing 7.5 -> 8 (Polymer-Familie identifiziert)

KEIN .kicad_pcb. PR #35 ist jetzt review-ready: 9 Commits von r18.5 bis
r18.12 plus Repo-Phase-1-Refactor, 12 ADRs, alle Schematic-Validierungen
gruen. Empfehlung: PR mergen und r18.13 mit Repo-Refactor Phase 2 (Doc-
Moves) oder Firmware-HAL-Abstraktion starten.

https://claude.ai/code/session_01K5kLTFpDCCoYwx2dq6Rk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
Parts:
- EN1, EN2, EN3, EN4: footprint Rotary_Encoder:RotaryEncoder_Alps_EC11E-Switch_Vertical_H20mm -> field_ambience:RotaryEncoder_ALPS_EC11J_SMD; FP_DRAFT (none) -> field_ambience:RotaryEncoder_ALPS_EC11J_SMD ist ein DRAFT-F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; FP_VERIFY F-2: KiCad-Standard-FP ist EC11E (THT-Stems); EC11J ist SMD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 -> (none)
Changed lines of the file:
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@@
       (property "Value" "EC11 + push (DRIVE)" (at 142.54 71.27 0)
         (effects (font (size 1.27 1.27))))
-      (property "Footprint" "Rotary_Encoder:RotaryEncoder_Alps_EC11E-Switch_Vertical_H20mm" (at 140.0 70 0)
+      (property "Footprint" "field_ambience:RotaryEncoder_ALPS_EC11J_SMD" (at 140.0 70 0)
         (effects (font (size 1.27 1.27)) hide))
       (property "Datasheet" "https://jlcpcb.com/partdetail/C209762" (at 140.0 70 0)
@@
       (property "Status" "NRND (ALPS marks as Not Recommended For New Designs) — Prototype-OK, Serie: Ersatztyp wählen" (at 142.54 78.89 0)
         (effects (font (size 1.27 1.27)) hide))
-      (property "FP_VERIFY" "F-2: KiCad-Standard-FP ist EC11E (THT-Stems); EC11J ist SMD-Bauform. Vor Layout Land-Pattern gegen JLCPCB-EasyEDA-Drawing für C209762 abgleichen oder eigenen FP zeichnen." (at 142.54 80.16 0)
+      (property "FP_DRAFT" "field_ambience:RotaryEncoder_ALPS_EC11J_SMD ist ein DRAFT-FP aus den dokumentierten ALPS-EC11J-Standard-Maßen (12x13.4mm Body, 2.5mm Pad-Pitch). Vor Fab gegen EasyEDA-Export von C209762 verifizieren (jlcpcb.com/partdetail/ALPSALPINE-EC11J1525402/C209762 → Footprint-Download → KiCad-Import) und ggf. nachbessern." (at 142.54 80.16 0)
         (effects (font (size 1.27 1.27)) hide))
     (instances
@@
       (property "Value" "EC11 + push (BRIGHT)" (at 142.54 106.27 0)
         (effects (font (size 1.27 1.27))))
-      (property "Footprint" "Rotary_Encoder:RotaryEncoder_Alps_EC11E-Switch_Vertical_H20mm" (at 140.0 105 0)
+      (property "Footprint" "field_ambience:RotaryEncoder_ALPS_EC11J_SMD" (at 140.0 105 0)
         (effects (font (size 1.27 1.27)) hide))
       (property "Datasheet" "https://jlcpcb.com/partdetail/C209762" (at 140.0 105 0)
@@
       (property "Status" "NRND (ALPS marks as Not Recommended For New Designs) — Prototype-OK, Serie: Ersatztyp wählen" (at 142.54 113.89 0)
         (effects (font (size 1.27 1.27)) hide))
-      (property "FP_VERIFY" "F-2: KiCad-Standard-FP ist EC11E (THT-Stems); EC11J ist SMD-Bauform. Vor Layout Land-Pattern gegen JLCPCB-EasyEDA-Drawing für C209762 abgleichen oder eigenen FP zeichnen." (at 142.54 115.16 0)
+      (property "FP_DRAFT" "field_ambience:RotaryEncoder_ALPS_EC11J_SMD ist ein DRAFT-FP aus den dokumentierten ALPS-EC11J-Standard-Maßen (12x13.4mm Body, 2.5mm Pad-Pitch). Vor Fab gegen EasyEDA-Export von C209762 verifizieren (jlcpcb.com/partdetail/ALPSALPINE-EC11J1525402/C209762 → Footprint-Download → KiCad-Import) und ggf. nachbessern." (at 142.54 115.16 0)
         (effects (font (size 1.27 1.27)) hide))
     (instances
@@
       (property "Value" "EC11 + push (DISPLAY)" (at 142.54 141.27 0)
         (effects (font (size 1.27 1.27))))
-      (property "Footprint" "Rotary_Encoder:RotaryEncoder_Alps_EC11E-Switch_Vertical_H20mm" (at 140.0 140 0)
+      (property "Footprint" "field_ambience:RotaryEncoder_ALPS_EC11J_SMD" (at 140.0 140 0)
         (effects (font (size 1.27 1.27)) hide))
       (property "Datasheet" "https://jlcpcb.com/partdetail/C209762" (at 140.0 140 0)
@@
       (property "Status" "NRND (ALPS marks as Not Recommended For New Designs) — Prototype-OK, Serie: Ersatztyp wählen" (at 142.54 148.89 0)
         (effects (font (size 1.27 1.27)) hide))
-      (property "FP_VERIFY" "F-2: KiCad-Standard-FP ist EC11E (THT-Stems); EC11J ist SMD-Bauform. Vor Layout Land-Pattern gegen JLCPCB-EasyEDA-Drawing für C209762 abgleichen oder eigenen FP zeichnen." (at 142.54 150.16 0)
+      (property "FP_DRAFT" "field_ambience:RotaryEncoder_ALPS_EC11J_SMD ist ein DRAFT-FP aus den dokumentierten ALPS-EC11J-Standard-Maßen (12x13.4mm Body, 2.5mm Pad-Pitch). Vor Fab gegen EasyEDA-Export von C209762 verifizieren (jlcpcb.com/partdetail/ALPSALPINE-EC11J1525402/C209762 → Footprint-Download → KiCad-Import) und ggf. nachbessern." (at 142.54 150.16 0)
         (effects (font (size 1.27 1.27)) hide))
     (instances
@@
       (property "Value" "EC11 + push (VOL)" (at 142.54 176.27 0)
         (effects (font (size 1.27 1.27))))
-      (property "Footprint" "Rotary_Encoder:RotaryEncoder_Alps_EC11E-Switch_Vertical_H20mm" (at 140.0 175 0)
+      (property "Footprint" "field_ambience:RotaryEncoder_ALPS_EC11J_SMD" (at 140.0 175 0)
         (effects (font (size 1.27 1.27)) hide))
       (property "Datasheet" "https://jlcpcb.com/partdetail/C209762" (at 140.0 175 0)
@@
       (property "Status" "NRND (ALPS marks as Not Recommended For New Designs) — Prototype-OK, Serie: Ersatztyp wählen" (at 142.54 183.89 0)
         (effects (font (size 1.27 1.27)) hide))
-      (property "FP_VERIFY" "F-2: KiCad-Standard-FP ist EC11E (THT-Stems); EC11J ist SMD-Bauform. Vor Layout Land-Pattern gegen JLCPCB-EasyEDA-Drawing für C209762 abgleichen oder eigenen FP zeichnen." (at 142.54 185.16 0)
-        (effects (font (size 1.27 1.27)) hide))
-    (instances
+      (property "FP_DRAFT" "field_ambience:RotaryEncoder_ALPS_EC11J_SMD ist ein DRAFT-FP aus den dokumentierten ALPS-EC11J-Standard-Maßen (12x13.4mm Body, 2.5mm Pad-Pitch). Vor Fab gegen EasyEDA-Export von C209762 verifizieren (jlcpcb.com/partdetail/ALPSALPINE-EC11J1525402/C209762 → Footprint-Download → KiCad-Import) und ggf. nachbessern." (at 142.54 185.16 0)
+        (effects (font (size 1.27 1.27)) hide))
+    (instances
