File: field-ambience-current/kicad/battery.kicad_sch (KiCad schematic)
At the start: 22 parts, among them J9 JST PH 2.0 2-pin (LiPo Batter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, Q1 DMG2305UX P-MOS SOT-23 (USB-C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, U7 MCP73831T-2ACI/OT (LiPo Charg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, U8 TPS61089RNR (Boost LiPo→5V, 2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

Commit message: pcb(r18.6): Engineering-Verifikation — AP7361C-Pinout-Fix, TPS61089-Quelle, Custom-FP, BOM-LCSC, ADR-MIDI
Reaktion auf User-Korrekturen aus öffentlichen Datasheets. Vier
🔴-Blocker geschlossen, einer auf eine Design-Entscheidung umklassifiziert.

=== AP7361A-Pinout war FALSCH — gefixt + AP7361C ===

r18.5-Annahme: 1=ADJ/NC, 2=OUT, 3=IN, 4=GND, 5=EN.
Korrekt (Diodes-DS via mouser.de/datasheet/3/175/1/AP7361.pdf,
User-verifiziert):
    1=EN, 2=GND, 3=ADJ/NC, 4=IN, 5=OUT

Hätte zu einem totem Board geführt (IN/OUT/EN vertauscht).

Zusätzlich:
- Symbol auf AP7361C umbenannt (Diodes markiert AP7361 als NRND ->
  use AP7361C; gleicher SOT-89-5-Pinout)
- AP7361C-33Y5-13 = LCSC C460397 (SOT-89-5) statt r18.5-Kandidat
  C150719 (= SOT-223, falsches Package; verworfen)
- Cin/Cout 4.7 µF X5R 0603 (DS-Empfehlung, statt 1µF/2.2µF)
- Symbol-Pinmap + power_tree-Verdrahtung umgebaut: EN-Pin liegt
  jetzt links oben (statt links unten), IN links unten, OUT
  rechts oben — neu gerechnete Stub-Wires + Junctions

=== TPS61089-Footprint + Datenblatt-Anchor ===

- Symbol-Pinmap (1=FSW … 11=SW) verifiziert gegen TI Rev C Tabelle 6-1
  (User-Quelle ti.com/lit/gpn/tps61089) — als PIN_SOURCE-Property
- Footprint-Name auf RNR0011A-Konvention 2.0x2.5mm VQFN-HR
- RNSR-PDF → datasheets/legacy/TPS61089RNSR_wrong_variant.pdf

=== Encoder C209762 (NRND, Prototype-OK) ===

- MPN EC11J1525402, LCSC C209762 (JLCPCB-verifiziert)
- Datasheet-Link auf JLCPCB-Detail-Seite (ALPS-Drawing nicht öffentlich)
- Status: NRND als Property — Prototype-OK, Serie braucht Ersatztyp
- FP_VERIFY-Hinweis (EC11J ist SMD, der KiCad-Standard-FP EC11E ist THT)

=== Custom-Footprint für HX 12x12 (SW6-10) ===

- libraries/field_ambience.pretty/SW_HX_12x12x7.3_SMD-4P.kicad_mod
  basierend auf LCSC-Daten von C36498966:
  - SMD-4P, 11.8x11.8mm Body, 7.3mm Höhe
  - 4 Pads je 2.5x1.5mm auf 7mm-Pitch (X+Y)
  - SPST: gegenüberliegende Pads verbunden (1↔1, 2↔2)
  - Silkscreen + Pin-1-Dot + Courtyard +0.25mm IPC-7351B
- fp-lib-table um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
Parts:
- U8: footprint Package_DFN_QFN:VQFN-11-1EP_2.6x2.6mm_P0.5mm_EP0.85x1.5mm_HotRod -> Package_DFN_QFN:VQFN-HR-11-1EP_2x2.5mm_P0.4mm_EP0.7x1.4mm; FP_VERIFY (none) -> RNR0011A-Land-Pattern (2.0x2.5mm VQFN-HR) muss vor Layout g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; Manufacturer (none) -> Texas Instruments; PIN_SOURCE (none) -> TI-Datenblatt TPS61089 Rev C, Pin Functions Tabelle 6-1: 1=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; Package (none) -> VQFN-HR 11-pin 2.0 x 2.5 mm (RNR0011A)
Changed lines of the file:
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@@
       (property "Value" "TPS61089RNR (Boost LiPo→5V, 2A, programmable Fsw)" (at 142.54 91.27 0)
         (effects (font (size 1.27 1.27))))
-      (property "Footprint" "Package_DFN_QFN:VQFN-11-1EP_2.6x2.6mm_P0.5mm_EP0.85x1.5mm_HotRod" (at 140.0 90.0 0)
+      (property "Footprint" "Package_DFN_QFN:VQFN-HR-11-1EP_2x2.5mm_P0.4mm_EP0.7x1.4mm" (at 140.0 90.0 0)
         (effects (font (size 1.27 1.27)) hide))
       (property "Datasheet" "https://www.ti.com/lit/ds/symlink/tps61089.pdf" (at 140.0 90.0 0)
@@
       (property "MPN" "TPS61089RNR" (at 142.54 93.81 0)
         (effects (font (size 1.27 1.27)) hide))
-      (property "LCSC" "C165129" (at 142.54 95.08 0)
+      (property "Manufacturer" "Texas Instruments" (at 142.54 95.08 0)
+        (effects (font (size 1.27 1.27)) hide))
+      (property "LCSC" "C165129" (at 142.54 96.35 0)
+        (effects (font (size 1.27 1.27)) hide))
+      (property "Package" "VQFN-HR 11-pin 2.0 x 2.5 mm (RNR0011A)" (at 142.54 97.62 0)
+        (effects (font (size 1.27 1.27)) hide))
+      (property "PIN_SOURCE" "TI-Datenblatt TPS61089 Rev C, Pin Functions Tabelle 6-1: 1=FSW, 2=VCC, 3=FB, 4=COMP, 5=GND, 6=VOUT, 7=EN, 8=ILIM, 9=VIN, 10=BOOT, 11=SW (Symbol entspricht dem)" (at 142.54 98.89 0)
+        (effects (font (size 1.27 1.27)) hide))
+      (property "FP_VERIFY" "RNR0011A-Land-Pattern (2.0x2.5mm VQFN-HR) muss vor Layout gegen TI-Datenblatt Mechanical Drawing geprueft werden; aktueller FP-Name ist Annahme bzgl. KiCad-Standard-Lib" (at 142.54 100.16 0)
         (effects (font (size 1.27 1.27)) hide))
     (instances

Commit message: pcb(r18.7): ADR-0005 Phase-5-Gate gestrichen + FP_VERIFY-Pass (6 von 9 gelöst)
User: "Es muss da drauf laufen können. Weil warum nicht? Mach einfach
weiter. Es ist ja sowieso besser als pico 2."

Pragmatischer Call. ADR-0005 dokumentiert ehrlich:
- RP2350 trägt Engine bereits, H743 hat 3-4× CPU-Headroom + FPU +
  dedizierte SAI/TIM-QEI-Peripherie
- Erwarteter CPU-Bedarf ~10-15 %, weit unter 40 %-Gate
- Worst-Case: ein Prototyp-Spin mit reduzierter Funktionalität,
  nicht totes Board
- Layout-Pfad jetzt: ERC → FP_VERIFY → Layout (Hardware-Profiling
  läuft parallel, nicht sequenziell)

Folgedokumente aktualisiert: PROJECT_STATUS, PROJECT_MAP, ADR-0003,
PCB_LAYOUT_STATUS.

=== FP_VERIFY-Pass — 6 von 9 closed ===

| Position           | Lösung                                            |
|--------------------|---------------------------------------------------|
| U1 LQFP-100        | KiCad-Standard verifiziert (JEDEC MS-026)         |
| U5 SOT-89-5        | KiCad-Standard verifiziert (JEDEC TO-243)         |
| Y1 HC-49/US        | Custom-FP nach ABRACON-DS (5.6×2.1 mm @ 9.5)      |
| U8 TPS61089RNR     | Custom-FP nach TI Mech. Drawing 4222143/A         |
| Q2 2N7002 SOT-23   | KiCad-Standard verifiziert (JEDEC TO-236)         |
| J3 LCD-Header      | KiCad-Standard verifiziert (2.54 mm 1×8)          |
| EN1-4 EC11J        | Bleibt offen — ALPS-Drawing nicht öffentlich      |

KiCad-Standard-FPs wurden direkt vom kicad-footprints@master-Repo
raw-geprüft (Pad-Coords, Pitch, Courtyard).

=== Custom-Footprints ===

kicad/libraries/field_ambience.pretty/ jetzt 3 FPs:
- SW_HX_12x12x7.3_SMD-4P            (r18.6, HX-Button)
- Crystal_HC49-US-SMD_ABLS          (r18.7, ABLS-Crystal)
- Texas_VQFN-HR-11_2x2.5mm_P0.5mm_RNR0011A  (r18.7, TPS61089RNR)

ABLS-Custom war nötig weil KiCad-Standard Crystal_SMD_HC49-SD nur
4.5×2.0 mm Pads @ 8.5 mm Pitch hat — ABRACON empfiehlt 5.6×2.1 mm
@ 9.5 mm (Page 3 Drawing 450669 Rev AD). Funktional ginge der KiCad-
Standard auch, aber die ABRACON-S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
Parts:
- U8: footprint Package_DFN_QFN:VQFN-HR-11-1EP_2x2.5mm_P0.4mm_EP0.7x1.4mm -> field_ambience:Texas_VQFN-HR-11_2x2.5mm_P0.5mm_RNR0011A; FP_NOTE (none) -> Custom-FP field_ambience:Texas_VQFN-HR-11_2x2.5mm_P0.5mm_RN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; FP_VERIFY RNR0011A-Land-Pattern (2.0x2.5mm VQFN-HR) muss vor Layout g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 -> (none)
Connections:
- net GND: no longer U8.12 (ePAD)
Changed lines of the file:
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@@
       (property "Value" "TPS61089RNR (Boost LiPo→5V, 2A, programmable Fsw)" (at 142.54 91.27 0)
         (effects (font (size 1.27 1.27))))
-      (property "Footprint" "Package_DFN_QFN:VQFN-HR-11-1EP_2x2.5mm_P0.4mm_EP0.7x1.4mm" (at 140.0 90.0 0)
+      (property "Footprint" "field_ambience:Texas_VQFN-HR-11_2x2.5mm_P0.5mm_RNR0011A" (at 140.0 90.0 0)
         (effects (font (size 1.27 1.27)) hide))
       (property "Datasheet" "https://www.ti.com/lit/ds/symlink/tps61089.pdf" (at 140.0 90.0 0)
@@
       (property "PIN_SOURCE" "TI-Datenblatt TPS61089 Rev C, Pin Functions Tabelle 6-1: 1=FSW, 2=VCC, 3=FB, 4=COMP, 5=GND, 6=VOUT, 7=EN, 8=ILIM, 9=VIN, 10=BOOT, 11=SW (Symbol entspricht dem)" (at 142.54 98.89 0)
         (effects (font (size 1.27 1.27)) hide))
-      (property "FP_VERIFY" "RNR0011A-Land-Pattern (2.0x2.5mm VQFN-HR) muss vor Layout gegen TI-Datenblatt Mechanical Drawing geprueft werden; aktueller FP-Name ist Annahme bzgl. KiCad-Standard-Lib" (at 142.54 100.16 0)
+      (property "FP_NOTE" "Custom-FP field_ambience:Texas_VQFN-HR-11_2x2.5mm_P0.5mm_RNR0011A — TI-RNR0011A Land Pattern (Datasheet Mechanical Drawing 4222143/A, 08/2015) nachgebaut: 8x Side-Pads 0.55x0.25mm @ 0.5mm Pitch, EP-Pads 5+6 je 0.7x1.0mm, EP 11 (Thermal Pad) zentral 2.35x0.7mm. Alternative: TPS61089RNRR-FP von UltraLibrarian direkt importieren." (at 142.54 100.16 0)
         (effects (font (size 1.27 1.27)) hide))
     (instances
@@
       (project "field_ambience"
         (path "/f6a664dc-7032-4108-a10b-e4076008e6bd" (reference "#PWR_R_ILIM") (unit 1)))))
-  (symbol (lib_id "Power:GND") (at 140.0 101.43 0) (unit 1)
-    (in_bom yes) (on_board yes) (dnp no)
-      (property "Reference" "#PWR_U8_EPAD" (at 142.54 98.89 0)
-        (effects (font (size 1.27 1.27))))
-      (property "Value" "GND" (at 142.54 102.7 0)
-        (effects (font (size 1.27 1.27))))
-      (property "Footprint" "" (at 140.0 101.43 0)
-        (effects (font (size 1.27 1.27)) hide))
-      (property "Datasheet" "~" (at 140.0 101.43 0)
-        (effects (font (size 1.27 1.27)) hide))
-    (instances
-      (project "field_ambience"
-        (path "/f6a664dc-7032-4108-a10b-e4076008e6bd" (reference "#PWR_U8_EPAD") (unit 1)))))
   (symbol (lib_id "Device:C") (at 180 105 0) (unit 1)
     (in_bom yes) (on_board yes) (dnp no)
@@
     (stroke (width 0) (type default))
 )
-  (wire (pts (xy 140.0 98.89) (xy 140.0 101.43))
-    (stroke (width 0) (type default))
-)

Commit message: pcb(r18.20c): L1 Phantom-FP-Fix + Stale-STEPs cleanup
🟠 HIGH — L1 SWPA6045 hatte Phantom-Footprint-Name
Generator referenzierte Inductor_SMD:L_0630_6.0x6.0mm — existiert in
KiCad-Standard-Lib NICHT. PCB-Export wäre fehlgeschlagen oder hätte einen
leeren Footprint angenommen. Beim Footprint-Coverage-Scan gefunden.

Fix: EasyEDA-verifizierten Footprint für C83455 (war seit r18.14-3D-Aktion
in /tmp/3dfetch/ verfügbar) als field_ambience:L_Sunlord_SWPA6045 in
Project-Lib vendored. 2 SMD-Pads 2.2×5.72mm @ 5mm Pitch.

🟡 LOW — Stale STEPs entfernt
- SW-SMD_EC11J1525402-H24.5.step (EC11J retired r18.14)
- TYPE-C-SMD_6P-H3.2.step (M-17 retired r18.19)
MANIFEST.md aktualisiert (beide als retired, USB-C-C165948-Regen als TODO).

Custom-FPs: 5 → 7. Schematic-Footprint-Coverage: 0 Phantom-FPs verbleiben.

8/8 paren-balanced, Firmware 13/13 PASS.

Files: generate_kicad_project.py, libraries/field_ambience.pretty/
L_Sunlord_SWPA6045.kicad_mod NEU, battery.kicad_sch regen, FP_VERIFY_LOG,
BOM_MASTER, mechanical/3d_models/MANIFEST.

https://claude.ai/code/session_01K5kLTFpDCCoYwx2dq6RkAv
Parts:
- L1: footprint Inductor_SMD:L_0630_6.0x6.0mm -> field_ambience:L_Sunlord_SWPA6045
Changed lines of the file:
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@@
       (property "Value" "2.2uH 5A Shielded 0630 (TPS61089 Boost Inductor)" (at 142.54 76.27 0)
         (effects (font (size 1.27 1.27))))
-      (property "Footprint" "Inductor_SMD:L_0630_6.0x6.0mm" (at 140 75 0)
+      (property "Footprint" "field_ambience:L_Sunlord_SWPA6045" (at 140 75 0)
         (effects (font (size 1.27 1.27)) hide))
       (property "Datasheet" "~" (at 140 75 0)
