File: field-ambience-current/kicad/stm32h743.kicad_sch (KiCad schematic)
At the start: 45 parts, among them J4 SWD 1.27mm (SWCLK/GND/SWDIO), U1 STM32H743VIT6 (480MHz M7, LQF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, Y1 8MHz ABLS-8.000MHZ-B4-T (CL=1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

Commit message: pcb(r18.20b): Sourcing-Fills — alle JLC-bestückbaren TBD-LCSC geschlossen
Sourcing-Agent lieferte verifizierte in-Stock-LCSC für alle r18.20-TBDs:
- C_HSE1/2:  C107045 (Yageo 27pF C0G/NP0 0603, JLC Basic, ~834k Stock)
- C_BULK:    C444831 (Kyocera AVX TPSE477K010R0100, 470µF/10V Polymer Case-E)
- C_BULK2:   C2880380 (Taiyo Yuden 100µF/10V 1210)
- LED gelb:  C2287 (Hubei KENTO KT-0603Y, Vf 2.4V) — Hold + 5 Cell
- LED grün:  C12624 (Hubei KENTO KT-0603G pure-green, Vf 3.1V) — Shift + 5 Cell

Engineering-Flag 1: "220µF/10V/1210 existiert nicht" (220µF nur bis 6.3V im
1210). Statt 220µF/6.3V (am 5V-Rail auf ~70-110µF derated) → 100µF/10V mit
echtem Headroom. Effektiv-Bulk vergleichbar, audit-sauber.

Engineering-Flag 2: <25mΩ-Flach-Polymer (Panasonic SVPF/Kemet T520) bei LCSC
nicht lagernd. Bester JLC-Flach-Polymer C444831 (100mΩ). Verfehlt 10mΩ-Ziel,
aber paralleler 100µF-MLCC (~5mΩ) dominiert Transient-Impedanz → Bulk-ESR
unkritisch. Footprint Case-D→Case-E (7343-43, 4.3mm, passt in 8mm-Top-Zone).

Beifang: BOM_MASTER §9 sagte "220Ω LED-R", Generator sagt 390Ω (an +5V-Anode
→ LED → PCA9685-Sink). 5V/390Ω: gelb 6.7mA, grün 4.9mA — beide im 2-8mA-
Fenster, Wert bleibt. BOM_MASTER korrigiert.

Verifizierung: 8/8 paren-balanced, 0 TBD-VERIFY-Leftovers in power_tree+mcp,
LED gelb ×6 + grün ×6, Firmware 13/13 PASS.

Files: generate_kicad_project.py (5 Fills), 3 Sheets regen, BOM_MASTER,
ADR-0011 (ESR-Realität), CHANGELOG, PROJECT_QUALITY BOM 9.5→10, Readiness 6.5→7.

https://claude.ai/code/session_01K5kLTFpDCCoYwx2dq6RkAv
Parts:
- C_HSE1, C_HSE2: LCSC TBD-r18.20 (27pF C0G/NP0 50V 0603 — Sourcing-Agent) -> C107045; NOTE (none) -> 27pF C0G/NP0 50V 0603, JLC Basic, ~834k Stock (r18.20b veri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; VERIFY-STOCK 27pF +-5% C0G/NP0 50V 0603; vorher 22pF/C1804 (zu klein, C_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 -> (none)
Changed lines of the file:
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@@
       (property "Manufacturer" "Yageo" (at 95.54 207.43 0)
         (effects (font (size 1.27 1.27)) hide))
-      (property "LCSC" "TBD-r18.20 (27pF C0G/NP0 50V 0603 — Sourcing-Agent)" (at 95.54 208.7 0)
+      (property "LCSC" "C107045" (at 95.54 208.7 0)
         (effects (font (size 1.27 1.27)) hide))
-      (property "VERIFY-STOCK" "27pF +-5% C0G/NP0 50V 0603; vorher 22pF/C1804 (zu klein, C_stray-Annahme 7pF)" (at 95.54 209.97 0)
+      (property "NOTE" "27pF C0G/NP0 50V 0603, JLC Basic, ~834k Stock (r18.20b verifiziert). Vorher 22pF/C1804 (zu klein, implizierte C_stray=7pF). Final bench-tuned am OSC_OUT." (at 95.54 209.97 0)
         (effects (font (size 1.27 1.27)) hide))
     (instances
@@
       (property "Manufacturer" "Yageo" (at 109.54 207.43 0)
         (effects (font (size 1.27 1.27)) hide))
-      (property "LCSC" "TBD-r18.20 (27pF C0G/NP0 50V 0603 — Sourcing-Agent)" (at 109.54 208.7 0)
+      (property "LCSC" "C107045" (at 109.54 208.7 0)
         (effects (font (size 1.27 1.27)) hide))
-      (property "VERIFY-STOCK" "27pF +-5% C0G/NP0 50V 0603; vorher 22pF/C1804 (zu klein, C_stray-Annahme 7pF)" (at 109.54 209.97 0)
+      (property "NOTE" "27pF C0G/NP0 50V 0603, JLC Basic, ~834k Stock (r18.20b verifiziert). Vorher 22pF/C1804 (zu klein, implizierte C_stray=7pF). Final bench-tuned am OSC_OUT." (at 109.54 209.97 0)
         (effects (font (size 1.27 1.27)) hide))
     (instances

Commit message: pcb(r18.24): 3 Verifikations-Punkte geschlossen — weiße-LED-Package, VREF+-Caps, ADC-Channels
Aus "gibt es noch offene Fragen" die 3 autonom lösbaren Punkte abgeräumt.

🟠 Weiße-LED-Package-Bug (neu gefunden via Live-Check):
LED_HB hatte MPN XL-1608UWC-04 (0603) + 0603-Footprint, aber LCSC C965818 =
XL-2012UWC = 0805-Teil. Package-Mismatch. Fix: C965808 (echtes 0603, 2.5M
Stock). BOM_MASTER hatte auch die 3 Modifier-Weiß-LEDs auf C965818 → gefixt.

🟠 VREF+ Decoupling (Audit-Punkt 5):
VREF+ (Pin 20) war nur an VDDA_3V3, kein dedizierter Cap am Pin. Ergänzt
C_VREF1 (1µF) + C_VREF2 (100nF) → GND (ST-Empfehlung). Reduziert ADC-Jitter
der Hall-Velocity.

🟢 ADC-Channels DS-bestätigt (Audit-Punkt 4):
ST-PDF via Distrelec-Mirror geparst: PA4=ADC12_INP18, PB0=ADC12_INP9,
PB1=ADC12_INP5 verbatim aus DS12110; PC0=ADC123_INP10, PC1=ADC123_INP11.
Alle 5 auf ADC1 → Scan-Mode. SPEC §5.6a auf "DS-bestätigt" hochgestuft.

8/8 paren-balanced, C_VREF1/2 present, Firmware 13/13 PASS.

Files: generate_kicad_project.py, stm32h743.kicad_sch regen, SPEC §5.6a,
BOM_MASTER, CHANGELOG.

https://claude.ai/code/session_01K5kLTFpDCCoYwx2dq6RkAv
Parts:
- added C_VREF1: 1uF X5R 0603 (VREF+ ref-decoupling), Capacitor_SMD:C_0603_1608Metric, symbol Device:C
- added C_VREF2: 100nF X7R 0603 (VREF+ HF), Capacitor_SMD:C_0603_1608Metric, symbol Device:C
- LED_HB: LCSC C965818 -> C965808
Connections:
- net GND: now also C_VREF1.2, C_VREF2.2
- net VDDA_3V3: now also C_VREF1.1, C_VREF2.1
Changed lines of the file:
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@@
       (project "field_ambience"
         (path "/e3bc855f-ca21-4bea-a5ff-d24a556f7f9e" (reference "#PWR_U1_VSSA") (unit 1)))))
+  (symbol (lib_id "Device:C") (at 105.14 88.09 0) (unit 1)
+    (in_bom yes) (on_board yes) (dnp no)
+      (property "Reference" "C_VREF1" (at 107.68 85.55 0)
+        (effects (font (size 1.27 1.27))))
+      (property "Value" "1uF X5R 0603 (VREF+ ref-decoupling)" (at 107.68 89.36 0)
+        (effects (font (size 1.27 1.27))))
+      (property "Footprint" "Capacitor_SMD:C_0603_1608Metric" (at 105.14 88.09 0)
+        (effects (font (size 1.27 1.27)) hide))
+      (property "Datasheet" "~" (at 105.14 88.09 0)
+        (effects (font (size 1.27 1.27)) hide))
+      (property "MPN" "CL10A105KB8NNNC" (at 107.68 91.9 0)
+        (effects (font (size 1.27 1.27)) hide))
+      (property "LCSC" "C15849" (at 107.68 93.17 0)
+        (effects (font (size 1.27 1.27)) hide))
+    (instances
+      (project "field_ambience"
+        (path "/e3bc855f-ca21-4bea-a5ff-d24a556f7f9e" (reference "C_VREF1") (unit 1)))))
+  (symbol (lib_id "Power:GND") (at 105.14 94.28 0) (unit 1)
+    (in_bom yes) (on_board yes) (dnp no)
+      (property "Reference" "#PWR_CVREF1" (at 107.68 91.74 0)
+        (effects (font (size 1.27 1.27))))
+      (property "Value" "GND" (at 107.68 95.55 0)
+        (effects (font (size 1.27 1.27))))
+      (property "Footprint" "" (at 105.14 94.28 0)
+        (effects (font (size 1.27 1.27)) hide))
+      (property "Datasheet" "~" (at 105.14 94.28 0)
+        (effects (font (size 1.27 1.27)) hide))
+    (instances
+      (project "field_ambience"
+        (path "/e3bc855f-ca21-4bea-a5ff-d24a556f7f9e" (reference "#PWR_CVREF1") (unit 1)))))
+  (symbol (lib_id "Device:C") (at 99.14 88.09 0) (unit 1)
+    (in_bom yes) (on_board yes) (dnp no)
+      (property "Reference" "C_VREF2" (at 101.68 85.55 0)
+        (effects (font (size 1.27 1.27))))
+      (property "Value" "100nF X7R 0603 (VREF+ HF)" (at 101.68 89.36 0)
+        (effects (font (size 1.27 1.27))))
+      (property "Footprint" "Capacitor_SMD:C_0603_1608Metric" (at 99.14 88.09 0)
+        (effects (font (size 1.27 1.27)) hide))
+      (property "Datasheet" "~" (at 99.14 88.09 0)
+        (effects (font (size 1.27 1.27)) hide))
+      (property "MPN" "CC0603KRX7R9BB104" (at 101.68 91.9 0)
+        (effects (font (size 1.27 1.27)) hide))
+      (property "LCSC" "C14663" (at 101.68 93.17 0)
+        (effects (font (size 1.27 1.27)) hide))
+    (instances
+      (project "field_ambience"
+        (path "/e3bc855f-ca21-4bea-a5ff-d24a556f7f9e" (reference "C_VREF2") (unit 1)))))
+  (symbol (lib_id "Power:GND") (at 99.14 94.28 0) (unit 1)
+    (in_bom yes) (on_board yes) (dnp no)
+      (property "Reference" "#PWR_CVREF2" (at 101.68 91.74 0)
+        (effects (font (size 1.27 1.27))))
+      (property "Value" "GND" (at 101.68 95.55 0)
+        (effects (font (size 1.27 1.27))))
+      (property "Footprint" "" (at 99.14 94.28 0)
+        (effects (font (size 1.27 1.27)) hide))
+      (property "Datasheet" "~" (at 99.14 94.28 0)
+        (effects (font (size 1.27 1.27)) hide))
+    (instances
+      (project "field_ambience"
+        (path "/e3bc855f-ca21-4bea-a5ff-d24a556f7f9e" (reference "#PWR_CVREF2") (unit 1)))))
   (symbol (lib_id "Device:Ferrite_Bead") (at 96.0 218.0 90) (unit 1)
     (in_bom yes) (on_board yes) (dnp no)
@@
       (property "MPN" "XL-1608UWC-04" (at 232.54 233.62 0)
         (effects (font (size 1.27 1.27)) hide))
-      (property "LCSC" "C965818" (at 232.54 234.89000000000001 0)
+      (property "LCSC" "C965808" (at 232.54 234.89000000000001 0)
         (effects (font (size 1.27 1.27)) hide))
     (instances
@@
     (stroke (width 0) (type default))
 )
+  (wire (pts (xy 112.14 84.28) (xy 105.14 84.28))
+    (stroke (width 0) (type default))
+)
+  (wire (pts (xy 105.14 91.9) (xy 105.14 94.28))
+    (stroke (width 0) (type default))
+)
+  (wire (pts (xy 112.14 84.28) (xy 99.14 84.28))
+    (stroke (width 0) (type default))
+)
+  (wire (pts (xy 99.14 91.9) (xy 99.14 94.28))
+    (stroke (width 0) (type default))
+)
   (wire (pts (xy 147.62 61.42) (xy 142.62 61.42))
     (stroke (width 0) (type default))
@@
     (stroke (width 0) (type default))
 )
+  (junction (at 105.14 84.28) (diameter 0) (color 0 0 0 0)
+)
   (junction (at 102.0 218.0) (diameter 0) (color 0 0 0 0)
