File: field-ambience-current/kicad/stm32h743.kicad_sch (KiCad schematic)
At the start: 35 parts, among them J10 3.5mm TRS MIDI-Out (Type A, P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, J4 SWD 1.27mm (SWCLK/GND/SWDIO), U1 STM32H743VIT6 (480MHz M7, LQF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, Y1 8MHz ABLS-8.000MHZ-B4-T (CL=1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

Commit message: fix(pcb): geometric pin-level ERC — 7 copper shorts, 4 open circuits, boost loop instability (r18.80) (#92)
Headless geometric ERC (every pin anchor vs every wire segment, union-find
net build, hier-label/root-pin matching) over all 7 sheets found 12 real
defects; each verified in generator source and fixed there.

Copper shorts (pin/label anchors landing on foreign wires):
- power_tree: USB D+ AND D- hard-shorted to +5V — the U5 LDO block sat in
  the USB data corridor (EN pin on the DP wire, IN pin on the DM wire,
  rail drop overlapping the ESD VBUS wire). Block moved to (130,130).
- mcp: I2C_SCL shorted to GND — C5's GND pin landed exactly on the SCL
  wire (VDD pin 9 and SCL pin 12 are exactly 3 grid rows = 7.62mm apart,
  the cap's pin pitch). Entire I2C bus (U2+U6+U10) was dead. C5/C5b moved.
- audio: PCM_XSMT and I2S_LRCK shorted to GND (same 7.62mm trap, C8a/C8b
  and C_LDOO) — DAC permanently muted / no word clock. Caps flipped up.
- stm32: BOOT0 permanently HIGH twice over (+3V3 flag placed on the BOOT0
  node point; SW_BOOT wire drawn through its own pin-2 anchor) — MCU would
  always enter the ROM bootloader, never firmware.
- stm32: VDDA copper-tied to VDD (pin-21 stub drawn through the VDD pin-100
  anchor), bypassing FB2.
- battery: U8_SW_NODE label sat on the SW/BOOT wire crossing, merging the
  bootstrap net with the switch node (C_BOOT ineffective).

Open circuits:
- lcd: J3 LCD header — all 8 pins floating (wiring assumed KiCad-standard
  pins at -5.08 left; custom lib has pins at +3.81 right). J3 rotated 180.
- stm32: J4 SWD header — all 3 pins floating (same assumption). Board was
  unprogrammable.
- stm32: FB2 rotated 90 off its wires — both pins floating (VDDA had no
  intended supply path).
- stm32: lib_symbols entry lacked the MCU: prefix — KiCad cannot resolve
  U1 at all (exact lib_id match required).

Boost control loop (TPS61089, TI SLVSD38C eqs 15/17/18, validated by
reproducing TI's own 9V/2A reference values):
- R_COMP 22k -> 6.2k (n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
Parts:
- C_VDD1A, C_VDD2A, C_VDD3A, C_VDD4A, C_VDD5A: value 4.7uF X5R 0805 10V (VDD bulk) -> 22uF X5R 0805 25V (VDD bulk; r18.80: C45783=CL21A226MAQNNNE, 4.7uF-Angabe war falsch); MPN CL21A475KQFNNNE -> CL21A226MAQNNNE
Connections:
- net +3V3: now also FB2.1, U1.100 (VDD), U1.11 (VDD), U1.27 (VDD), U1.50 (VDD), U1.6 (VBAT), U1.75 (VDD); no longer R_BOOT0.1, R_BOOT_SW.1, SW_BOOT.1, SW_BOOT.2
- net AMP_nMUTE: now also U1.54 (PB15)
- net AMP_nSHDN: now also U1.53 (PB14)
- net BAT_SENSE: now also U1.25 (PA3)
- net BRIGHT_A: now also U1.63 (PC6)
- net BRIGHT_B: now also U1.64 (PC7)
- net BRIGHT_SW: now also U1.98 (PE1)
- net DISPLAY_A: now also U1.59 (PD12)
- net DISPLAY_B: now also U1.60 (PD13)
- net DISPLAY_SW: now also U1.2 (PE3)
- net DRIVE_A: now also U1.22 (PA0)
- net DRIVE_B: now also U1.23 (PA1)
- net DRIVE_SW: now also U1.97 (PE0)
- net GND: now also J4.2 (Pin_2), U1.10 (VSS), U1.19 (VSSA), U1.26 (VSS), U1.49 (VSS), U1.74 (VSS)
- net HSE_IN: now also U1.12 (PH0)
- net HSE_OUT: now also U1.13 (PH1)
- net I2C_SCL: now also U1.92 (PB6)
- net I2C_SDA: now also U1.93 (PB7)
- net I2S_BCK: now also U1.4 (PE5)
- net I2S_DOUT: now also U1.5 (PE6)
- net I2S_LRCK: now also U1.3 (PE4)
- net LCD_CS: now also U1.30 (PA6)
- net LCD_DC: now also U1.32 (PC4)
- net LCD_MOSI: now also U1.31 (PA7)
- net LCD_RES: now also U1.33 (PC5)
- net LCD_SCK: now also U1.29 (PA5)
- net MCP_INT: now also U1.7 (PC13)
- net MIDI_TX: now also U1.86 (PD5)
- net NC_PA4_ADC_RSVD: now also U1.28 (PA4)
- net NC_PB0_ADC_RSVD: now also U1.34 (PB0)
- net NC_PB1_ADC_RSVD: now also U1.35 (PB1)
- net NC_PC0_ADC_RSVD: now also U1.15 (PC0)
- net NC_PC1_ADC_RSVD: now also U1.16 (PC1)
- net NRST: now also U1.14 (NRST)
- net STATUS_LED: now also U1.55 (PD8)
- net SWCLK: now also J4.1 (Pin_1), U1.76 (PA14)
- net SWDIO: now also J4.3 (Pin_3), U1.72 (PA13)
- net SWO: now also U1.89 (PB3)
- net USB_DM: now also U1.70 (PA11)
- net USB_DP: now also U1.71 (PA12)
- net VDDA_3V3: now also FB2.2, U1.20 (VREF+), U1.21 (VDDA)
- net VOL_A: now also U1.67 (PA8)
- net VOL_B: now also U1.68 (PA9)
- net at C_VCAP2.1: now also U1.73 (VCAP2)
- net at C_VCAP1.1: now also U1.48 (VCAP1)
- new net: R_BOOT_SW.1, SW_BOOT.2
- new net BOOT0_PIN: R_BOOT0.1, SW_BOOT.1, U1.94 (BOOT0)
Other:
- moved on the sheet: FB2
Changed lines of the file:
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@@
       (project "field_ambience"
         (path "/e3bc855f-ca21-4bea-a5ff-d24a556f7f9e" (reference "#PWR_CVREF2") (unit 1)))))
-  (symbol (lib_id "Device:Ferrite_Bead") (at 96.0 218.0 90) (unit 1)
+  (symbol (lib_id "Device:Ferrite_Bead") (at 96.0 218.0 0) (unit 1)
     (in_bom yes) (on_board yes) (dnp no)
       (property "Reference" "FB2" (at 98.54 215.46 0)
@@
       (property "Reference" "C_VDD1A" (at 98.54 235.46 0)
         (effects (font (size 1.27 1.27))))
-      (property "Value" "4.7uF X5R 0805 10V (VDD bulk)" (at 98.54 239.27 0)
+      (property "Value" "22uF X5R 0805 25V (VDD bulk; r18.80: C45783=CL21A226MAQNNNE, 4.7uF-Angabe war falsch)" (at 98.54 239.27 0)
         (effects (font (size 1.27 1.27))))
       (property "Footprint" "Capacitor_SMD:C_0805_2012Metric" (at 96.0 238.0 0)
@@
       (property "Datasheet" "~" (at 96.0 238.0 0)
         (effects (font (size 1.27 1.27)) hide))
-      (property "MPN" "CL21A475KQFNNNE" (at 98.54 241.81 0)
+      (property "MPN" "CL21A226MAQNNNE" (at 98.54 241.81 0)
         (effects (font (size 1.27 1.27)) hide))
       (property "LCSC" "C45783" (at 98.54 243.08 0)
@@
       (property "Reference" "C_VDD2A" (at 110.54 235.46 0)
         (effects (font (size 1.27 1.27))))
-      (property "Value" "4.7uF X5R 0805 10V (VDD bulk)" (at 110.54 239.27 0)
+      (property "Value" "22uF X5R 0805 25V (VDD bulk; r18.80: C45783=CL21A226MAQNNNE, 4.7uF-Angabe war falsch)" (at 110.54 239.27 0)
         (effects (font (size 1.27 1.27))))
       (property "Footprint" "Capacitor_SMD:C_0805_2012Metric" (at 108.0 238.0 0)
@@
       (property "Datasheet" "~" (at 108.0 238.0 0)
         (effects (font (size 1.27 1.27)) hide))
-      (property "MPN" "CL21A475KQFNNNE" (at 110.54 241.81 0)
+      (property "MPN" "CL21A226MAQNNNE" (at 110.54 241.81 0)
         (effects (font (size 1.27 1.27)) hide))
       (property "LCSC" "C45783" (at 110.54 243.08 0)
@@
       (property "Reference" "C_VDD3A" (at 122.54 235.46 0)
         (effects (font (size 1.27 1.27))))
-      (property "Value" "4.7uF X5R 0805 10V (VDD bulk)" (at 122.54 239.27 0)
+      (property "Value" "22uF X5R 0805 25V (VDD bulk; r18.80: C45783=CL21A226MAQNNNE, 4.7uF-Angabe war falsch)" (at 122.54 239.27 0)
         (effects (font (size 1.27 1.27))))
       (property "Footprint" "Capacitor_SMD:C_0805_2012Metric" (at 120.0 238.0 0)
@@
       (property "Datasheet" "~" (at 120.0 238.0 0)
         (effects (font (size 1.27 1.27)) hide))
-      (property "MPN" "CL21A475KQFNNNE" (at 122.54 241.81 0)
+      (property "MPN" "CL21A226MAQNNNE" (at 122.54 241.81 0)
         (effects (font (size 1.27 1.27)) hide))
       (property "LCSC" "C45783" (at 122.54 243.08 0)
@@
       (property "Reference" "C_VDD4A" (at 134.54 235.46 0)
         (effects (font (size 1.27 1.27))))
-      (property "Value" "4.7uF X5R 0805 10V (VDD bulk)" (at 134.54 239.27 0)
+      (property "Value" "22uF X5R 0805 25V (VDD bulk; r18.80: C45783=CL21A226MAQNNNE, 4.7uF-Angabe war falsch)" (at 134.54 239.27 0)
         (effects (font (size 1.27 1.27))))
       (property "Footprint" "Capacitor_SMD:C_0805_2012Metric" (at 132.0 238.0 0)
@@
       (property "Datasheet" "~" (at 132.0 238.0 0)
         (effects (font (size 1.27 1.27)) hide))
-      (property "MPN" "CL21A475KQFNNNE" (at 134.54 241.81 0)
+      (property "MPN" "CL21A226MAQNNNE" (at 134.54 241.81 0)
         (effects (font (size 1.27 1.27)) hide))
       (property "LCSC" "C45783" (at 134.54 243.08 0)
@@
       (property "Reference" "C_VDD5A" (at 146.54 235.46 0)
         (effects (font (size 1.27 1.27))))
-      (property "Value" "4.7uF X5R 0805 10V (VDD bulk)" (at 146.54 239.27 0)
+      (property "Value" "22uF X5R 0805 25V (VDD bulk; r18.80: C45783=CL21A226MAQNNNE, 4.7uF-Angabe war falsch)" (at 146.54 239.27 0)
         (effects (font (size 1.27 1.27))))
       (property "Footprint" "Capacitor_SMD:C_0805_2012Metric" (at 144.0 238.0 0)
@@
       (property "Datasheet" "~" (at 144.0 238.0 0)
         (effects (font (size 1.27 1.27)) hide))
-      (property "MPN" "CL21A475KQFNNNE" (at 146.54 241.81 0)
+      (property "MPN" "CL21A226MAQNNNE" (at 146.54 241.81 0)
         (effects (font (size 1.27 1.27)) hide))
       (property "LCSC" "C45783" (at 146.54 243.08 0)
@@
       (project "field_ambience"
         (path "/e3bc855f-ca21-4bea-a5ff-d24a556f7f9e" (reference "R_BOOT_SW") (unit 1)))))
-  (symbol (lib_id "Power:+3V3") (at 100.0 184.0 90) (unit 1)
-    (in_bom yes) (on_board yes) (dnp no)
-      (property "Reference" "#PWR_SWBOOT" (at 102.54 181.46 0)
-        (effects (font (size 1.27 1.27))))
-      (property "Value" "+3V3" (at 102.54 185.27 0)
-        (effects (font (size 1.27 1.27))))
-      (property "Footprint" "" (at 100.0 184.0 0)
-        (effects (font (size 1.27 1.27)) hide))
-      (property "Datasheet" "~" (at 100.0 184.0 0)
+  (symbol (lib_id "Power:+3V3") (at 98.81 180.0 0) (unit 1)
+    (in_bom yes) (on_board yes) (dnp no)
+      (property "Reference" "#PWR_SWBOOT" (at 101.35000000000001 177.46 0)
+        (effects (font (size 1.27 1.27))))
+      (property "Value" "+3V3" (at 101.35000000000001 181.27 0)
+        (effects (font (size 1.27 1.27))))
+      (property "Footprint" "" (at 98.81 180.0 0)
+        (effects (font (size 1.27 1.27)) hide))
+      (property "Datasheet" "~" (at 98.81 180.0 0)
         (effects (font (size 1.27 1.27)) hide))
     (instances
@@
       (project "field_ambience"
         (path "/e3bc855f-ca21-4bea-a5ff-d24a556f7f9e" (reference "J4") (unit 1)))))
-  (symbol (lib_id "Power:GND") (at 187.0 208.0 90) (unit 1)
-    (in_bom yes) (on_board yes) (dnp no)
-      (property "Reference" "#PWR_J4" (at 189.54 205.46 0)
-        (effects (font (size 1.27 1.27))))
-      (property "Value" "GND" (at 189.54 209.27 0)
-        (effects (font (size 1.27 1.27))))
-      (property "Footprint" "" (at 187.0 208.0 0)
-        (effects (font (size 1.27 1.27)) hide))
-      (property "Datasheet" "~" (at 187.0 208.0 0)
+  (symbol (lib_id "Power:GND") (at 205.0 208.0 270) (unit 1)
+    (in_bom yes) (on_board yes) (dnp no)
+      (property "Reference" "#PWR_J4" (at 207.54 205.46 0)
+        (effects (font (size 1.27 1.27))))
+      (property "Value" "GND" (at 207.54 209.27 0)
+        (effects (font (size 1.27 1.27))))
+      (property "Footprint" "" (at 205.0 208.0 0)
+        (effects (font (size 1.27 1.27)) hide))
+      (property "Datasheet" "~" (at 205.0 208.0 0)
         (effects (font (size 1.27 1.27)) hide))
     (instances
@@
     (stroke (width 0) (type default))
 )
-  (wire (pts (xy 147.62 61.42) (xy 142.62 61.42))
+  (wire (pts (xy 147.62 61.42) (xy 147.62 56.42))
     (stroke (width 0) (type default))
 )
@@
     (stroke (width 0) (type default))
 )
-  (wire (pts (xy 80.92 184.0) (xy 100.0 184.0))
+  (wire (pts (xy 80.92 184.0) (xy 80.92 190.0))
+    (stroke (width 0) (type default))
+)
+  (wire (pts (xy 80.92 190.0) (xy 100.0 190.0))
+    (stroke (width 0) (type default))
+)
+  (wire (pts (xy 100.0 190.0) (xy 100.0 184.0))
     (stroke (width 0) (type default))
 )
@@
     (stroke (width 0) (type default))
 )
-  (wire (pts (xy 98.81 184.0) (xy 100.0 184.0))
-    (stroke (width 0) (type default))
-)
-  (wire (pts (xy 190.92 205.46) (xy 187.0 205.46))
-    (stroke (width 0) (type default))
-)
-  (wire (pts (xy 190.92 210.54) (xy 187.0 210.54))
-    (stroke (width 0) (type default))
-)
-  (wire (pts (xy 190.92 208.0) (xy 187.0 208.0))
+  (wire (pts (xy 98.81 184.0) (xy 98.81 180.0))
+    (stroke (width 0) (type default))
+)
+  (wire (pts (xy 199.81 205.46) (xy 205.0 205.46))
+    (stroke (width 0) (type default))
+)
+  (wire (pts (xy 199.81 210.54) (xy 205.0 210.54))
+    (stroke (width 0) (type default))
+)
+  (wire (pts (xy 199.81 208.0) (xy 205.0 208.0))
     (stroke (width 0) (type default))
 )
@@
     (effects (font (size 1.27 1.27)) (justify left bottom))
 )
-  (label "VDDA_3V3" (at 142.62 61.42 0) (fields_autoplaced)
+  (label "VDDA_3V3" (at 147.62 56.42 90) (fields_autoplaced)
     (effects (font (size 1.27 1.27)) (justify left bottom))
 )
@@
     (effects (font (size 1.27 1.27)) (justify left bottom))
 )
-  (label "SWCLK" (at 187.0 205.46 0) (fields_autoplaced)
-    (effects (font (size 1.27 1.27)) (justify left bottom))
-)
-  (label "SWDIO" (at 187.0 210.54 0) (fields_autoplaced)
-    (effects (font (size 1.27 1.27)) (justify left bottom))
-)
+  (label "SWCLK" (at 205.0 205.46 0) (fields_autoplaced)
+    (effects (font (size 1.27 1.27)) (justify left bottom))
+)
+  (label "SWDIO" (at 205.0 210.54 0) (fields_autoplaced)
+    (effects (font (size 1.27 1.27)) (justify left bottom))
+)
